File: tr_sonde/$tr.sch (KiCad schematic (older format))
At the start: 100 parts, among them J1 SMA, J2 SMA, J3 SMA, K1 TR, K2 HV_MON, K3 VINHDR, Q1 PBSS4250X, Q2 MMBT2222A, Q3 STD2NK90ZT4, Q4 STD2NK90ZT4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

Commit message: updated tr board to remove DNP components
Parts:
- removed C14, C16, C19, C21: DNP, smd_capacitors:c_0805, symbol C
- removed C29: 100nF, smd_capacitors:c_0805, symbol C
- removed R10, R4, R5, R8, R9: 0, smd_capacitors:c_0805, symbol R
- removed R20, R23, R24, R26, R3: DNP, smd_capacitors:c_0805, symbol R
- removed U5: 74AHC1G04, SMD_Packages:SOT23-5, symbol 74AHC1G04
- C10: value 4700pF -> 4700pF 600V
- C15, C2, C6: value .022uF -> .022uF 600 V
- C30: value .47uF -> .47uF 600V
- C33: value 4700pF -> 4700pF 600 V
- C34: value .022uF -> .022uF 600V
- C5: value 68nF -> 68nF 600V
- C9: value .022uF -> .022uF, 600 V
- D9: value SMBJ250CACT-ND -> P6SMB550CA
- R18: value 2k2 -> 10k
Connections:
- net hvd is gone; now on net hvbias: Q4.D
- net hvout is gone; now on net hvbias: C5.2, U1.6 (OUT)
- net hvs is gone; now on net hvbias: Q3.S
- net RXDRV: now also R19.1
- net TX: now also D11.1 (A)
- net TXDRV: no longer R19.1
- net at U1.5 (LVG): now also Q4.G
- net at U1.7 (HVG): now also Q3.G
Other:
- moved on the sheet: D11, R11, R18
