File: mimic/mimic.sch (KiCad schematic (older format))
At the start: 60 parts, among them J1 SMA, J2 SMA, J3 SMA, J4 SMA, U1 XCO, U2 AD9835, U3 AD9835, U4 HMC595, U5 HMC595, U6 teensy_3.1

Commit message: added LPF on dds output and merged spi control lines on schematic
Parts:
- removed R23: 0, SMD_Packages:SM0603, symbol R
- removed R24: DNP, SMD_Packages:SM0603, symbol R
- R10, R13, R14, R9: value DNP -> 180 pF
- R11, R12: value 0 -> 820 nH
- R3, R4: value 300 -> DNP
Connections:
- net FSYNC1: now also U6.14 (12/DIN)
- net SCLK1 renamed SCLK
- net SCLK: now also U2.7 (SCLK)
- net SCLK2: no longer names the net of U6.4 (2/CS)
- net SCLK2: no longer U2.7 (SCLK)
- net SDATA1 renamed SDATA
- net SDATA: now also U2.8 (SDATA)
- net SDATA2: no longer names the net of U6.5 (3/TX)
- net SDATA2: no longer U2.8 (SDATA)
Changed lines of the file:
@@
 LIBS:ad9835
 LIBS:teensy_3
-LIBS:adp3338
 LIBS:xco
 LIBS:sma
@@
 P 4050 2850
 F 0 "R4" V 4130 2850 40  0000 C CNN
-F 1 "300" V 4057 2851 40  0000 C CNN
+F 1 "DNP" V 4057 2851 40  0000 C CNN
 F 2 "SMD_Packages:SM0603" V 3980 2850 30  0001 C CNN
 F 3 "" H 4050 2850 30  0000 C CNN
@@
 REFCLK
 Text Label 1550 2900 2    60   ~ 0
-SCLK1
+SCLK
 Text Label 1550 3000 2    60   ~ 0
-SDATA1
+SDATA
 $Comp
 L +5V #PWR011
@@
 P 5300 2500
 F 0 "R12" V 5380 2500 40  0000 C CNN
-F 1 "0" V 5307 2501 40  0000 C CNN
+F 1 "820 nH" V 5307 2501 40  0000 C CNN
 F 2 "SMD_Packages:SM0603" V 5230 2500 30  0001 C CNN
 F 3 "" H 5300 2500 30  0000 C CNN
@@
 P 5600 2850
 F 0 "R14" V 5680 2850 40  0000 C CNN
-F 1 "DNP" V 5607 2851 40  0000 C CNN
+F 1 "180 pF" V 5607 2851 40  0000 C CNN
 F 2 "SMD_Packages:SM0603" V 5530 2850 30  0001 C CNN
 F 3 "" H 5600 2850 30  0000 C CNN
@@
 P 5000 2850
 F 0 "R10" V 5080 2850 40  0000 C CNN
-F 1 "DNP" V 5007 2851 40  0000 C CNN
+F 1 "180 pF" V 5007 2851 40  0000 C CNN
 F 2 "SMD_Packages:SM0603" V 4930 2850 30  0001 C CNN
 F 3 "" H 5000 2850 30  0000 C CNN
@@
 P 4000 6650
 F 0 "R3" V 4080 6650 40  0000 C CNN
-F 1 "300" V 4007 6651 40  0000 C CNN
+F 1 "DNP" V 4007 6651 40  0000 C CNN
 F 2 "SMD_Packages:SM0603" V 3930 6650 30  0001 C CNN
 F 3 "" H 4000 6650 30  0000 C CNN
@@
 REFCLK
 Text Label 1500 6700 2    60   ~ 0
-SCLK2
+SCLK
 Text Label 1500 6800 2    60   ~ 0
-SDATA2
+SDATA
 $Comp
 L +5V #PWR027
@@
 P 5250 6300
 F 0 "R11" V 5330 6300 40  0000 C CNN
-F 1 "0" V 5257 6301 40  0000 C CNN
+F 1 "820 nH" V 5257 6301 40  0000 C CNN
 F 2 "SMD_Packages:SM0603" V 5180 6300 30  0001 C CNN
 F 3 "" H 5250 6300 30  0000 C CNN
@@
 P 5550 6650
 F 0 "R13" V 5630 6650 40  0000 C CNN
-F 1 "DNP" V 5557 6651 40  0000 C CNN
+F 1 "180 pF" V 5557 6651 40  0000 C CNN
 F 2 "SMD_Packages:SM0603" V 5480 6650 30  0001 C CNN
 F 3 "" H 5550 6650 30  0000 C CNN
@@
 P 4950 6650
 F 0 "R9" V 5030 6650 40  0000 C CNN
-F 1 "DNP" V 4957 6651 40  0000 C CNN
+F 1 "180 pF" V 4957 6651 40  0000 C CNN
 F 2 "SMD_Packages:SM0603" V 4880 6650 30  0001 C CNN
 F 3 "" H 4950 6650 30  0000 C CNN
@@
 	0    -1   -1   0
 $EndComp
-Text Label 11650 6700 2    60   ~ 0
+Text Label 11800 6800 2    60   ~ 0
 FSYNC2
-Text Label 11650 6800 2    60   ~ 0
+Text Label 11800 6900 2    60   ~ 0
 FSYNC1
 Text Label 11850 6600 2    60   ~ 0
-SDATA1
+SDATA
 Text Label 11850 6500 2    60   ~ 0
-SCLK1
-Text Label 11750 5900 2    60   ~ 0
-SCLK2
-Text Label 11750 6000 2    60   ~ 0
-SDATA2
-$Comp
-L R R23
-U 1 1 53A287AE
-P 12150 6800
-F 0 "R23" V 12230 6800 40  0000 C CNN
-F 1 "0" V 12157 6801 40  0000 C CNN
-F 2 "SMD_Packages:SM0603" V 12080 6800 30  0001 C CNN
-F 3 "" H 12150 6800 30  0000 C CNN
-	1    12150 6800
-	0    1    1    0
-$EndComp
-$Comp
-L R R24
-U 1 1 53A28C24
-P 12150 6900
-F 0 "R24" V 12230 6900 40  0000 C CNN
-F 1 "DNP" V 12157 6901 40  0000 C CNN
-F 2 "SMD_Packages:SM0603" V 12080 6900 30  0001 C CNN
-F 3 "" H 12150 6900 30  0000 C CNN
-	1    12150 6900
-	0    1    1    0
-$EndComp
+SCLK
 $Comp
 L R R17
@@
 Text Label 1700 8800 1    60   ~ 0
 REFEN
-Text Label 12600 6700 2    60   ~ 0
+Text Label 11800 6700 2    60   ~ 0
 REFEN
 $Comp
@@
 	4850 1550 4850 1450
 Wire Wire Line
-	12650 5900 11750 5900
-Wire Wire Line
 	5600 10100 5600 10150
 Wire Wire Line
@@
 	9400 2550 9300 2550
 Wire Wire Line
-	11750 6000 12650 6000
-Wire Wire Line
 	5600 8650 5600 8700
 Wire Wire Line
@@
 	5200 8050 5650 8050
 Wire Wire Line
-	11800 6900 11900 6900
-Wire Wire Line
-	12400 6900 12650 6900
-Connection ~ 12450 6800
-Wire Wire Line
-	12450 6700 12450 6800
-Wire Wire Line
-	12400 6800 12650 6800
-Connection ~ 11800 6800
-Wire Wire Line
-	11650 6800 11900 6800
-Wire Wire Line
-	11800 6900 11800 6800
-Wire Wire Line
-	11650 6700 12450 6700
+	11800 6900 12650 6900
 Wire Wire Line
 	12650 6500 11850 6500
@@
 Connection ~ 14850 6200
 Wire Wire Line
-	12600 6700 12650 6700
+	11800 6700 12650 6700
+Wire Wire Line
+	11800 6800 12650 6800
 $EndSCHEMATC
