File: tr/tr.sch (KiCad schematic (older format))
At the start: 105 parts, among them J1 SMA, J2 SMA, J3 SMA, K1 CONN_3, Q1 Si7850, Q3 STD2NK90ZT4, Q4 STD2NK90ZT4, T1 DA2033-AL_, U1 L6388E, U2 LT1631, U3 LT3757

Commit message: added connectors
Parts:
- added K?: CONN_3, ~, symbol CONN_3
Connections:
- net GND: now also K?.2 (PM)
- net VCC: now also K?.1 (P1)
- net VEE: now also K?.3 (P3)
Other:
- moved on the sheet: K1, R27, R28
Changed lines of the file:
@@
 L CONN_3 K1
 U 1 1 52ABD194
-P 18050 10650
-F 0 "K1" V 18000 10650 50  0000 C CNN
-F 1 "CONN_3" V 18100 10650 40  0000 C CNN
-F 2 "~" H 18050 10650 60  0000 C CNN
-F 3 "~" H 18050 10650 60  0000 C CNN
-	1    18050 10650
+P 18050 8000
+F 0 "K1" V 18000 8000 50  0000 C CNN
+F 1 "CONN_3" V 18100 8000 40  0000 C CNN
+F 2 "~" H 18050 8000 60  0000 C CNN
+F 3 "~" H 18050 8000 60  0000 C CNN
+	1    18050 8000
 	1    0    0    -1
 $EndComp
@@
 L GND #PWR017
 U 1 1 52ABD1A1
-P 17200 10650
-F 0 "#PWR017" H 17200 10650 30  0001 C CNN
-F 1 "GND" H 17200 10580 30  0001 C CNN
-F 2 "" H 17200 10650 60  0000 C CNN
-F 3 "" H 17200 10650 60  0000 C CNN
-	1    17200 10650
+P 17200 8000
+F 0 "#PWR017" H 17200 8000 30  0001 C CNN
+F 1 "GND" H 17200 7930 30  0001 C CNN
+F 2 "" H 17200 8000 60  0000 C CNN
+F 3 "" H 17200 8000 60  0000 C CNN
+	1    17200 8000
 	0    1    1    0
 $EndComp
-Text Label 17250 10550 0    60   ~ 0
+Text Label 17250 7900 0    60   ~ 0
 RX
-Text Label 17250 10750 0    60   ~ 0
+Text Label 17250 8100 0    60   ~ 0
 TX
 $Comp
@@
 TX
 $Comp
-L R R27
-U 1 1 52AF509C
-P 17500 10150
-F 0 "R27" V 17580 10150 40  0000 C CNN
-F 1 "20k" V 17507 10151 40  0000 C CNN
-F 2 "~" V 17430 10150 30  0000 C CNN
-F 3 "~" H 17500 10150 30  0000 C CNN
-	1    17500 10150
-	-1   0    0    1
-$EndComp
-$Comp
 L R R28
 U 1 1 52AF50A2
-P 17500 11150
-F 0 "R28" V 17580 11150 40  0000 C CNN
-F 1 "20k" V 17507 11151 40  0000 C CNN
-F 2 "~" V 17430 11150 30  0000 C CNN
-F 3 "~" H 17500 11150 30  0000 C CNN
-	1    17500 11150
+P 17500 8500
+F 0 "R28" V 17580 8500 40  0000 C CNN
+F 1 "20k" V 17507 8501 40  0000 C CNN
+F 2 "~" V 17430 8500 30  0000 C CNN
+F 3 "~" H 17500 8500 30  0000 C CNN
+	1    17500 8500
 	-1   0    0    1
 $EndComp
@@
 L GND #PWR035
 U 1 1 52AF534D
-P 17500 9750
-F 0 "#PWR035" H 17500 9750 30  0001 C CNN
-F 1 "GND" H 17500 9680 30  0001 C CNN
-F 2 "" H 17500 9750 60  0000 C CNN
-F 3 "" H 17500 9750 60  0000 C CNN
-	1    17500 9750
+P 17500 7100
+F 0 "#PWR035" H 17500 7100 30  0001 C CNN
+F 1 "GND" H 17500 7030 30  0001 C CNN
+F 2 "" H 17500 7100 60  0000 C CNN
+F 3 "" H 17500 7100 60  0000 C CNN
+	1    17500 7100
 	-1   0    0    1
 $EndComp
@@
 L GND #PWR037
 U 1 1 52AF5793
-P 17500 11600
-F 0 "#PWR037" H 17500 11600 30  0001 C CNN
-F 1 "GND" H 17500 11530 30  0001 C CNN
-F 2 "" H 17500 11600 60  0000 C CNN
-F 3 "" H 17500 11600 60  0000 C CNN
-	1    17500 11600
+P 17500 8950
+F 0 "#PWR037" H 17500 8950 30  0001 C CNN
+F 1 "GND" H 17500 8880 30  0001 C CNN
+F 2 "" H 17500 8950 60  0000 C CNN
+F 3 "" H 17500 8950 60  0000 C CNN
+	1    17500 8950
 	1    0    0    -1
 $EndComp
@@
 	8150 9250 8150 9750
 Wire Wire Line
-	17700 10650 17200 10650
-Wire Wire Line
-	17200 10550 17700 10550
-Wire Wire Line
-	17200 10750 17700 10750
+	17700 8000 17200 8000
+Wire Wire Line
+	17200 7900 17700 7900
+Wire Wire Line
+	17200 8100 17700 8100
 Wire Wire Line
 	6600 3950 6600 4450
@@
 	11350 13200 11350 13500
 Wire Wire Line
-	17500 10400 17500 10550
-Connection ~ 17500 10550
-Wire Wire Line
-	17500 10750 17500 10900
-Connection ~ 17500 10750
+	17500 7750 17500 7900
+Connection ~ 17500 7900
+Wire Wire Line
+	17500 8100 17500 8250
+Connection ~ 17500 8100
 Wire Wire Line
 	19300 10800 19300 11000
 Wire Wire Line
-	17500 9900 17500 9750
+	17500 7250 17500 7100
 Wire Wire Line
 	19300 10200 19300 10400
 Wire Wire Line
-	17500 11400 17500 11600
+	17500 8750 17500 8950
 Wire Wire Line
 	18800 10800 18800 11000
@@
 	6100 13550 6100 13700
 Wire Wire Line
-	2650 12750 6850 12750
+	6850 12750 2650 12750
 Wire Wire Line
 	6100 12750 6100 13150
@@
 Connection ~ 3700 12750
 Wire Wire Line
-	5400 14750 5400 15150
+	5400 15150 5400 14750
 Connection ~ 4650 15150
 Wire Wire Line
@@
 	8800 14500 8800 15000
 Wire Wire Line
-	8800 15500 8800 15700
+	8800 15700 8800 15500
 Wire Wire Line
 	6150 15700 9450 15700
@@
 Text Notes 3100 10550 0    60   ~ 0
 todo: optocouple inputs? isolate power supply? overdesign other aspects?
+$Comp
+L CONN_3 K?
+U 1 1 53376FD9
+P 18000 6250
+F 0 "K?" V 17950 6250 50  0000 C CNN
+F 1 "CONN_3" V 18050 6250 40  0000 C CNN
+F 2 "~" H 18000 6250 60  0000 C CNN
+F 3 "~" H 18000 6250 60  0000 C CNN
+	1    18000 6250
+	1    0    0    -1
+$EndComp
+$Comp
+L GND #PWR?
+U 1 1 53376FDF
+P 17150 6250
+F 0 "#PWR?" H 17150 6250 30  0001 C CNN
+F 1 "GND" H 17150 6180 30  0001 C CNN
+F 2 "" H 17150 6250 60  0000 C CNN
+F 3 "" H 17150 6250 60  0000 C CNN
+	1    17150 6250
+	0    1    1    0
+$EndComp
+Wire Wire Line
+	17650 6250 17150 6250
+$Comp
+L R R27
+U 1 1 52AF509C
+P 17500 7500
+F 0 "R27" V 17580 7500 40  0000 C CNN
+F 1 "20k" V 17507 7501 40  0000 C CNN
+F 2 "~" V 17430 7500 30  0000 C CNN
+F 3 "~" H 17500 7500 30  0000 C CNN
+	1    17500 7500
+	-1   0    0    1
+$EndComp
+$Comp
+L VCC #PWR?
+U 1 1 5337703B
+P 17500 5750
+F 0 "#PWR?" H 17500 5850 30  0001 C CNN
+F 1 "VCC" H 17500 5850 30  0000 C CNN
+F 2 "" H 17500 5750 60  0000 C CNN
+F 3 "" H 17500 5750 60  0000 C CNN
+	1    17500 5750
+	1    0    0    -1
+$EndComp
+Wire Wire Line
+	17500 5750 17500 6150
+$Comp
+L VEE #PWR?
+U 1 1 53377042
+P 17500 6450
+F 0 "#PWR?" H 17500 6650 40  0001 C CNN
+F 1 "VEE" H 17500 6600 40  0000 C CNN
+F 2 "" H 17500 6450 60  0000 C CNN
+F 3 "" H 17500 6450 60  0000 C CNN
+	1    17500 6450
+	-1   0    0    1
+$EndComp
+Wire Wire Line
+	17500 6150 17650 6150
+Wire Wire Line
+	17650 6350 17500 6350
+Wire Wire Line
+	17500 6350 17500 6450
 $EndSCHEMATC

Commit message: started on t/r with enclosure, migrated distro to 15v
Parts:
- removed C12, C8: 10nF, ~, symbol C
- removed C14, C16, C19, C21: 100pF, 0805, symbol C
- removed C29, C33: 47uF, SM1210, symbol CAPAPOL
- removed D10: ES2A, SMB, symbol DIODE
- removed D11: ES2G-E3/52T, ~, symbol DIODE
- removed K?: CONN_3, ~, symbol CONN_3
- removed L2: 22uH, ~, symbol INDUCTOR
- removed Q1: Si7850, ~, symbol MOS_N_PPAK
- removed R10: 150, 0805, symbol R
- removed R15: RVAR, SM1210, symbol RVAR
- removed R20, R23, R24, R26: 22, 0805, symbol R
- removed R21: 330, 0805, symbol R
- removed R32: 105k, SM0603, symbol R
- removed R33, R35: 22, SM0603, symbol R
- removed R34: .02, SM0603, symbol R
- removed R36: 1.5M, SM0603, symbol R
- removed R37, R38: 1M, SM0603, symbol R
- removed R39: 16.2k, SM0603, symbol R
- removed R4, R5: 1k, 0805, symbol R
- removed R40: 1M, SM1210, symbol R
- removed R8, R9: 0, 0805, symbol R
- removed T1: DA2033-AL_, ~, symbol TRANSFO_MULTI
- removed U2: LT1631, ~, symbol LT1631
- removed U3: LT3757, ~, symbol LT3757
- added C12: 22uF, Capacitors_SMD:c_1210, symbol CAPAPOL
- added C33: 4700pF 600 V, SMD_Packages:SMD-1210, symbol C
- added D10: RED, LEDs:LED-0805, symbol LED
- added D11: GREEN, LEDs:LED-0805, symbol LED
- added F1: PTC FUSE (0ZCJ0010FF2E), Fuse_Holders_and_Fuses:Fuse_SMD1206_HandSoldering, symbol FUSE
- added K2: HV_MON, Connect:PINHEAD1-3, symbol CONN_3
- added K3: VINHDR, Connect:PINHEAD1-3, symbol CONN_3
- added K4: TR, Connect:PINHEAD1-3, symbol CONN_3
- added L7, L9: 10uH, Inductors:SELF-WE-TPC_M, symbol INDUCTOR
- added L8: 22uH, smd_capacitors:c_1210, symbol INDUCTOR
- added Q1: PBSS4250X, Transistors_SMD:sot89, symbol NPN_E1
- added Q2: MMBT2222A, SMD_Packages:SOT23EBC, symbol NPN
- added U2: 75451, SOIC_Packages:SOIC-8_N, symbol 7545x
- added U3: 5SA400, PICOPSU:xxSAxxxx, symbol xxSAxxxx
- C1, C17, C20, C3, R13, R2: footprint 0805 -> smd_capacitors:c_0805
- C10: value .022uF -> 4700pF 600V; footprint SM1210 -> smd_capacitors:c_1210
- C11, C7, C9: value .022uF -> .022uF, 600 V; footprint 1210 -> smd_capacitors:c_1210
- C13: value 2.2uF -> 100nF; footprint ~ -> smd_capacitors:c_0805
- C15, C2, C6: value .022uF -> .022uF 600 V; footprint 1210 -> smd_capacitors:c_1210
- C18, L1, L3, L4, L5, L6: footprint ~ -> smd_capacitors:c_1210
- C22, C23, R1, R12, R18, R19: footprint ~ -> smd_capacitors:c_0805
- C24: value 10uF -> 22uF; footprint ~ -> smd_capacitors:c_1210
- C25, C27, C31: value 47uF -> 22uF; footprint SM1210 -> smd_capacitors:c_1210
- C26: value 100pF -> 100nF; footprint SM0603 -> smd_capacitors:c_0805
- C28: value 22nF -> 100pF; footprint SM0603 -> smd_capacitors:c_0805
- C30: value 100nF -> .47uF 600V; footprint SM0603 -> Capacitors_SMD:c_2225
- C32: footprint SM0603 -> smd_capacitors:c_0805
- C34: value 220pF -> .022uF 600V; footprint 0805 -> SMD_Packages:SMD-1210
- C35: value 68nF -> 10nF; footprint SM1210 -> smd_capacitors:c_0805; DIGIKEYPN C3225X7R2J683K -> (none)
- C36: value 68nF -> 2.2uF; footprint SM1210 -> smd_capacitors:c_0805; DIGIKEYPN C3225X7R2J683K -> (none)
- C4: value 2.2uF -> 10nF; footprint ~ -> smd_capacitors:c_0805
- C5: value 68nF -> 68nF 600V; footprint 0805 -> SMD_Packages:SMD-1210
- D1, D6, D7, D8: footprint SMB -> smb_diode:SMB_DO2144AA
- D12: value ES2G-E3/52T -> ES2A; footprint ~ -> smb_diode:SMB_DO2144AA
- D2, D4: footprint MELF-1072 -> Diodes_SMD:Diode-SMB_Handsoldering
- D3, D5: footprint MELF-1072 -> melf-1072:MELF-1072
- D9: value ES2A -> P6SMB550CA; footprint SMB -> smb_diode:SMB_DO2144AA
- J1, J2, J3: footprint ~ -> sma:sma
- K1: value CONN_3 -> TR; footprint ~ -> Connect:PINHEAD1-3
- Q3, Q4: footprint TO-252-3 -> to252:TO252-3
- R11, R22: value 470 -> 150; footprint 0805 -> SMD_Packages:SMD-1210
- R14: value 10k -> 10M (HV, eg. HVC1206T1005JET); footprint ~ -> SMD_Packages:SM1210
- R16: value 20k -> 5k1; footprint ~ -> smd_capacitors:c_0805
- R17, R27, R28: value 20k -> 10k; footprint ~ -> smd_capacitors:c_0805
- R25: value 470 -> 220; footprint 0805 -> SMD_Packages:SMD-1210
- R29: value 6.8k -> 510; footprint SM0603 -> smd_capacitors:c_0805
- R3: value 10k -> 1k (500V+, eg HVCB1206JDD1K00); footprint ~ -> SMD_Packages:SM1210
- R30: value 140k -> 220; footprint SM0603 -> SMD_Packages:SMD-1210
- R31: value 46.4k -> 22; footprint SM0603 -> smd_capacitors:c_0805
- R6, R7: value 20k -> 300 (1W); footprint ~ -> smd_capacitors:c_1210
- U1: footprint S0-8 -> smd_dil:so-8
Connections:
- net OUTA is gone; now on net VCC: R6.2
- net VEE is gone; now on net +5V: C13.1
- net hvd is gone; now on net hvbias: Q4.D
- net hvout is gone; now on net hvbias: C5.2, U1.6 (OUT)
- net hvs is gone; now on net hvbias: Q3.S
- net GND: now also C26.2, C28.2, C3.2, C30.2, C34.2, C35.2, C36.2, D9.2 (K), R12.2, R17.2, R18.1, C12.2, C33.2, K2.3 (P3), K3.2 (PM), K4.2 (PM), Q2.1 (E), U2.4 (GND), U3.1 (IN-), U3.6 (-OUT); no longer C26.1, C28.1, C3.1, C30.1, C34.1, C35.1, C36.1, R12.1, R14.1, R27.2, R30.1
- net RX: now also U1.1 (LIN), U2.1 (1A), U2.2 (2B); no longer D9.1 (A), R1.1, R19.2
- net TX: now also U1.2 (HIN), D11.1 (A), U2.6 (2A), U2.7 (2B); no longer R18.2, R3.1
- net VCC: now also D12.2 (K), R29.1, R30.1, R7.2, D10.1 (A), L7.2; no longer C25.1, C27.1, C31.1, C4.1
- net VDD: now also C30.1, R14.2, R3.1
- net at U1.5 (LVG): now also Q4.G
- net at U1.7 (HVG): now also Q3.G
- net at C6.2, J2.1 (RF): now also D9.1 (A)
- net at C15.2, D2.1 (A): now also L8.2
- net at R16.2: now also C3.1, R14.1, K2.1 (P1); no longer R18.1
- net at R1.2: now also U3.2 (SHDN); no longer R6.1
- net at R3.2: now also C34.1, C33.1, K4.3 (P3), U3.4 (+OUT); no longer R7.1
- net RXDRV: now reaches R19.1
- net RXDRV: now also R11.1, R22.1, R6.1, U2.3 (1Y); no longer R17.2
- net at R29.2: now also Q1.3 (B), Q2.3 (C); no longer C26.2
- net at R30.2: now also C31.1, R31.1
- net at R31.2: now also Q1.2 (C)
- net at C32.2: now also L8.1, Q1.1 (E)
- net +5V: now reaches D12.1 (A)
- net +5V: now also C26.1, C35.1, C36.1, R27.2, C12.1, F1.1, L9.2, U2.8 (Vcc)
- removed net OUTB: R22.1, R7.2
- net OUTC: no longer names the net of R17.1
- net OUTC: now also C4.1, R16.1, K2.2 (PM); no longer R11.1
- net OUTD renamed TXDRV
- net TXDRV: now also R7.1, U2.5 (2Y); no longer R16.1
- new net: C25.1, C27.1, C28.1, F1.2, R1.1, U3.3 (+IN)
- new net: K3.1 (P1), L7.1
- new net: D10.2 (K), R12.1
- new net: D11.2 (K), R18.2
- new net: Q2.2 (B), R19.2
- new net: K3.3 (P3), L9.1
Other:
- note added: "400V Power Supply\n"
- note added: "aux 400V input (for off-board supplies)"
- note added: "trip at 300 mA, nominal 200 mA"
- note removed: "20 mA on\n"
- note removed: "20 mA on\n\n"
- note removed: "300V Power Supply\n"
- note removed: "40 mA on\n"
- note removed: "replace with 634U?\n"
- note removed: "todo: optocouple inputs? isolate power supply? overdesign other aspects?"
- moved on the sheet: C1, C10, C11, C15, C17, C18, C2, C20, C22, C23, C24, C25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
