File: agc/agc.sch (KiCad schematic (older format))
At the start: 112 parts, among them J1 SMA_DAC, J2 SMA_LPTR, J3 SMA_DRIVER, J4 SMA_RX, J5 SIL10, J6 SMA_LPTR, K1 TR, K3 VIN, K5 TR, K7 HVMON, P10 CONN_2, P2 FWD_FAULT, P3 REF_FAULT, P4 CONN_8X2, P5 COUPLED_TEST, P6 TP_VCC, P7 COUPLED_TEST, P8 COUPLED_TEST, P9 COUPLED_TEST, U1 BA08CC0WFP, U10 74AHC1G04, U11 74AHC1G04, U12 78SRH-5/2-C, U14 SMP1330-005LF, U15 SMP1330-005LF, U16 SMP1330-005LF, U2 HMC475, U3 HMC595, U4 HMC595, U5 HMC595, U6 74AHC1G04, U7 ISL3281E, U8 MGA-61563, U9 LTC2914-2

Commit message: polishing agc, tr, and driver amp for next revisions. moved all bottom layer signal traces to top layer on driver amp
Parts:
- removed R50: 0, SMD_Packages:SM0805, symbol R
- added K2: TR, Connect:PINHEAD1-3, symbol CONN_3
- C13, C14, C4: value 1nF -> 10nF
- C20: value 1.2pF -> DNP
- C28: value .1uF -> 10nF
- L4: value 1.2nH -> JMP
- R46, R47, R48, R49: value 1k -> 4k7
- gave numbers to parts that had none: 2
Connections:
- net GND: now also K2.2 (PM)
- net TX: now also K2.1 (P1)
- net ~TX: now also U10.4, U6.2, K2.3 (P3)
Other:
- note added: "TMR capacitor, 9ms/nF\n"
- note added: "to driver amplifier"
- note added: "to monitor"
- note removed: "INPUT +/- 15V"
- note removed: "vpp: 300V rail (20mA max)\nvcc: +15V rail (1500 mA max?)\nvee: -15V rail (200 mA max?)\n5v: +5V rail (150 mA max?)"
- moved on the sheet: K1, K5, P10
Changed lines of the file:
@@
 P 9800 2550
 F 0 "L4" H 9800 2650 50  0000 C CNN
-F 1 "1.2nH" H 9800 2500 50  0000 C CNN
+F 1 "JMP" H 9800 2500 50  0000 C CNN
 F 2 "SMD_Packages:SM0805" H 9800 2550 60  0001 C CNN
 F 3 "" H 9800 2550 60  0000 C CNN
@@
 P 9400 2850
 F 0 "C20" H 9400 2950 40  0000 L CNN
-F 1 "1.2pF" H 9406 2765 40  0000 L CNN
+F 1 "DNP" H 9406 2765 40  0000 L CNN
 F 2 "SMD_Packages:SM0805" H 9438 2700 30  0001 C CNN
 F 3 "" H 9400 2850 60  0000 C CNN
@@
 P 6850 7600
 F 0 "C14" H 6850 7700 40  0000 L CNN
-F 1 "1nF" H 6856 7515 40  0000 L CNN
+F 1 "10nF" H 6856 7515 40  0000 L CNN
 F 2 "SMD_Packages:SM0805" H 6888 7450 30  0001 C CNN
 F 3 "" H 6850 7600 60  0000 C CNN
@@
 P 6850 6650
 F 0 "C13" H 6850 6750 40  0000 L CNN
-F 1 "1nF" H 6856 6565 40  0000 L CNN
+F 1 "10nF" H 6856 6565 40  0000 L CNN
 F 2 "SMD_Packages:SM0805" H 6888 6500 30  0001 C CNN
 F 3 "" H 6850 6650 60  0000 C CNN
@@
 P 4150 6650
 F 0 "C4" H 4150 6750 40  0000 L CNN
-F 1 "1nF" H 4156 6565 40  0000 L CNN
+F 1 "10nF" H 4156 6565 40  0000 L CNN
 F 2 "SMD_Packages:SM0805" H 4188 6500 30  0001 C CNN
 F 3 "" H 4150 6650 60  0000 C CNN
@@
 	1    0    0    -1
 $EndComp
-Text Notes 950  11250 0    79   ~ 0
-INPUT +/- 15V
 $Comp
 L LTC2914 U9
@@
 P 19450 9650
 F 0 "C28" H 19450 9750 40  0000 L CNN
-F 1 ".1uF" H 19456 9565 40  0000 L CNN
+F 1 "10nF" H 19456 9565 40  0000 L CNN
 F 2 "SMD_Packages:SM0805" H 19488 9500 30  0001 C CNN
 F 3 "" H 19450 9650 60  0000 C CNN
@@
 	-1   0    0    1
 $EndComp
-Text Notes 18650 8450 0    79   ~ 0
+Text Notes 18150 9000 0    79   ~ 0
 FAULT DETECTION\n
 $Comp
@@
 P 7800 7500
 F 0 "R46" V 7880 7500 40  0000 C CNN
-F 1 "1k" V 7807 7501 40  0000 C CNN
+F 1 "4k7" V 7807 7501 40  0000 C CNN
 F 2 "SMD_Packages:SM0805" V 7730 7500 30  0001 C CNN
 F 3 "" H 7800 7500 30  0000 C CNN
@@
 P 8250 7500
 F 0 "R47" V 8330 7500 40  0000 C CNN
-F 1 "1k" V 8257 7501 40  0000 C CNN
+F 1 "4k7" V 8257 7501 40  0000 C CNN
 F 2 "SMD_Packages:SM0805" V 8180 7500 30  0001 C CNN
 F 3 "" H 8250 7500 30  0000 C CNN
@@
 	1    0    0    -1
 $EndComp
-Text Notes 1250 10700 0    79   ~ 0
-vpp: 300V rail (20mA max)\nvcc: +15V rail (1500 mA max?)\nvee: -15V rail (200 mA max?)\n5v: +5V rail (150 mA max?)
 Text Label 4200 5950 0    79   ~ 0
 FAULT
@@
 P 9500 13400
 F 0 "R49" V 9580 13400 40  0000 C CNN
-F 1 "1k" V 9507 13401 40  0000 C CNN
+F 1 "4k7" V 9507 13401 40  0000 C CNN
 F 2 "SMD_Packages:SM0805" V 9430 13400 30  0001 C CNN
 F 3 "" H 9500 13400 30  0000 C CNN
@@
 P 9500 12100
 F 0 "R48" V 9580 12100 40  0000 C CNN
-F 1 "1k" V 9507 12101 40  0000 C CNN
+F 1 "4k7" V 9507 12101 40  0000 C CNN
 F 2 "SMD_Packages:SM0805" V 9430 12100 30  0001 C CNN
 F 3 "" H 9500 12100 30  0000 C CNN
@@
 	1    0    0    -1
 $EndComp
-$Comp
-L R R50
-U 1 1 537CE1B1
-P 13550 12550
-F 0 "R50" V 13630 12550 40  0000 C CNN
-F 1 "0" V 13557 12551 40  0000 C CNN
-F 2 "SMD_Packages:SM0805" V 13480 12550 30  0001 C CNN
-F 3 "" H 13550 12550 30  0000 C CNN
-	1    13550 12550
-	0    -1   -1   0
-$EndComp
 Text Label 14100 12550 0    79   ~ 0
 ~TX
@@
 bypass for diff line driver\n
 NoConn ~ 1450 12200
-Text Label 15850 14650 0    79   ~ 0
+Text Label 15250 14650 0    79   ~ 0
 ~TX
-Text Label 15850 14850 0    79   ~ 0
+Text Label 15250 14850 0    79   ~ 0
 TX
 $Comp
 L CONN_3 K5
 U 1 1 537D1CD3
-P 15100 14750
-F 0 "K5" V 15050 14750 50  0000 C CNN
-F 1 "TR" V 15150 14750 40  0000 C CNN
-F 2 "Connect:PINHEAD1-3" H 15100 14750 60  0001 C CNN
-F 3 "" H 15100 14750 60  0000 C CNN
-	1    15100 14750
+P 14500 14750
+F 0 "K5" V 14450 14750 50  0000 C CNN
+F 1 "TR" V 14550 14750 40  0000 C CNN
+F 2 "Connect:PINHEAD1-3" H 14500 14750 60  0001 C CNN
+F 3 "" H 14500 14750 60  0000 C CNN
+	1    14500 14750
 	-1   0    0    1
 $EndComp
@@
 L GND #PWR059
 U 1 1 537D1CD9
-P 16150 14800
-F 0 "#PWR059" H 16150 14800 30  0001 C CNN
-F 1 "GND" H 16150 14730 30  0001 C CNN
-F 2 "" H 16150 14800 60  0000 C CNN
-F 3 "" H 16150 14800 60  0000 C CNN
-	1    16150 14800
-	1    0    0    -1
-$EndComp
-Text Label 15850 14200 0    79   ~ 0
+P 15550 14800
+F 0 "#PWR059" H 15550 14800 30  0001 C CNN
+F 1 "GND" H 15550 14730 30  0001 C CNN
+F 2 "" H 15550 14800 60  0000 C CNN
+F 3 "" H 15550 14800 60  0000 C CNN
+	1    15550 14800
+	1    0    0    -1
+$EndComp
+Text Label 15250 14200 0    79   ~ 0
 ~TX
-Text Label 15850 14400 0    79   ~ 0
+Text Label 15250 14400 0    79   ~ 0
 TX
 $Comp
 L CONN_3 K1
 U 1 1 537D1CE7
-P 15100 14300
-F 0 "K1" V 15050 14300 50  0000 C CNN
-F 1 "TR" V 15150 14300 40  0000 C CNN
-F 2 "Connect:PINHEAD1-3" H 15100 14300 60  0001 C CNN
-F 3 "" H 15100 14300 60  0000 C CNN
-	1    15100 14300
+P 14500 14300
+F 0 "K1" V 14450 14300 50  0000 C CNN
+F 1 "TR" V 14550 14300 40  0000 C CNN
+F 2 "Connect:PINHEAD1-3" H 14500 14300 60  0001 C CNN
+F 3 "" H 14500 14300 60  0000 C CNN
+	1    14500 14300
 	-1   0    0    1
 $EndComp
@@
 L GND #PWR060
 U 1 1 537D1CED
-P 16150 14350
-F 0 "#PWR060" H 16150 14350 30  0001 C CNN
-F 1 "GND" H 16150 14280 30  0001 C CNN
-F 2 "" H 16150 14350 60  0000 C CNN
-F 3 "" H 16150 14350 60  0000 C CNN
-	1    16150 14350
+P 15550 14350
+F 0 "#PWR060" H 15550 14350 30  0001 C CNN
+F 1 "GND" H 15550 14280 30  0001 C CNN
+F 2 "" H 15550 14350 60  0000 C CNN
+F 3 "" H 15550 14350 60  0000 C CNN
+	1    15550 14350
 	1    0    0    -1
 $EndComp
@@
 	12400 12750 12400 12850
 Wire Wire Line
-	12900 12550 13300 12550
-Wire Wire Line
-	13800 12550 14100 12550
+	12900 12550 14100 12550
 Wire Wire Line
 	11450 11600 11450 12750
@@
 	5300 9300 5300 9550
 Wire Wire Line
-	15450 14650 15850 14650
-Wire Wire Line
-	15450 14850 15850 14850
-Wire Wire Line
-	15450 14750 16150 14750
-Wire Wire Line
-	16150 14750 16150 14800
-Wire Wire Line
-	15450 14200 15850 14200
-Wire Wire Line
-	15450 14400 15850 14400
-Wire Wire Line
-	15450 14300 16150 14300
-Wire Wire Line
-	16150 14300 16150 14350
+	14850 14650 15250 14650
+Wire Wire Line
+	14850 14850 15250 14850
+Wire Wire Line
+	14850 14750 15550 14750
+Wire Wire Line
+	15550 14750 15550 14800
+Wire Wire Line
+	14850 14200 15250 14200
+Wire Wire Line
+	14850 14400 15250 14400
+Wire Wire Line
+	14850 14300 15550 14300
+Wire Wire Line
+	15550 14300 15550 14350
 Wire Wire Line
 	17600 8550 17600 8750
@@
 Text Label 6250 14350 1    79   ~ 0
 ~FAULT
-Text Notes 16500 14300 0    79   ~ 0
+Text Notes 15900 14300 0    79   ~ 0
 to T/R switch
-Text Notes 16500 14700 0    79   ~ 0
+Text Notes 15900 14700 0    79   ~ 0
 aux T/R output
 $Comp
 L CONN_2 P10
 U 1 1 53BDC57E
-P 16000 13600
-F 0 "P10" V 15950 13600 40  0000 C CNN
-F 1 "CONN_2" V 16050 13600 40  0000 C CNN
-F 2 "Connect:PINHEAD1-2" H 16000 13600 60  0001 C CNN
-F 3 "" H 16000 13600 60  0000 C CNN
-	1    16000 13600
+P 15300 13650
+F 0 "P10" V 15250 13650 40  0000 C CNN
+F 1 "CONN_2" V 15350 13650 40  0000 C CNN
+F 2 "Connect:PINHEAD1-2" H 15300 13650 60  0001 C CNN
+F 3 "" H 15300 13650 60  0000 C CNN
+	1    15300 13650
 	1    0    0    -1
 $EndComp
@@
 Text Label 13200 14600 0    79   ~ 0
 ~FAULT
-Text Label 15300 13500 2    79   ~ 0
+Text Label 14600 13550 2    79   ~ 0
 ~FAULT
 Wire Wire Line
-	15300 13500 15650 13500
+	14600 13550 14950 13550
 $Comp
 L GND #PWR085
 U 1 1 53BDCABB
-P 15300 13800
-F 0 "#PWR085" H 15300 13800 30  0001 C CNN
-F 1 "GND" H 15300 13730 30  0001 C CNN
-F 2 "" H 15300 13800 60  0000 C CNN
-F 3 "" H 15300 13800 60  0000 C CNN
-	1    15300 13800
-	1    0    0    -1
-$EndComp
-Wire Wire Line
-	15300 13800 15300 13700
-Wire Wire Line
-	15300 13700 15650 13700
+P 14600 13850
+F 0 "#PWR085" H 14600 13850 30  0001 C CNN
+F 1 "GND" H 14600 13780 30  0001 C CNN
+F 2 "" H 14600 13850 60  0000 C CNN
+F 3 "" H 14600 13850 60  0000 C CNN
+	1    14600 13850
+	1    0    0    -1
+$EndComp
+Wire Wire Line
+	14600 13850 14600 13750
+Wire Wire Line
+	14600 13750 14950 13750
 $Comp
 L SMA J6
@@
 	5250 1700 5350 1700
 $Comp
-L C C?
+L C C30
 U 1 1 53D18787
 P 16350 10750
-F 0 "C?" H 16350 10850 40  0000 L CNN
+F 0 "C30" H 16350 10850 40  0000 L CNN
 F 1 "10nF" H 16356 10665 40  0000 L CNN
 F 2 "SMD_Packages:SM0805" H 16388 10600 30  0001 C CNN
@@
 $EndComp
 $Comp
-L C C?
+L C C31
 U 1 1 53D18792
 P 16600 10750
-F 0 "C?" H 16600 10850 40  0000 L CNN
+F 0 "C31" H 16600 10850 40  0000 L CNN
 F 1 "10nF" H 16606 10665 40  0000 L CNN
 F 2 "SMD_Packages:SM0805" H 16638 10600 30  0001 C CNN
@@
 Connection ~ 16600 10150
 $Comp
-L GND #PWR?
+L GND #PWR093
 U 1 1 53D18C86
 P 16350 11050
-F 0 "#PWR?" H 16350 11050 30  0001 C CNN
+F 0 "#PWR093" H 16350 11050 30  0001 C CNN
 F 1 "GND" H 16350 10980 30  0001 C CNN
 F 2 "" H 16350 11050 60  0000 C CNN
@@
 	16600 10950 16600 11050
 $Comp
-L GND #PWR?
+L GND #PWR094
 U 1 1 53D18FD7
 P 16600 11050
-F 0 "#PWR?" H 16600 11050 30  0001 C CNN
+F 0 "#PWR094" H 16600 11050 30  0001 C CNN
 F 1 "GND" H 16600 10980 30  0001 C CNN
 F 2 "" H 16600 11050 60  0000 C CNN
@@
 	1    0    0    -1
 $EndComp
+Text Notes 19850 10050 0    39   ~ 0
+TMR capacitor, 9ms/nF\n
+Text Label 15250 15200 0    79   ~ 0
+~TX
+Text Label 15250 15400 0    79   ~ 0
+TX
+$Comp
+L CONN_3 K2
+U 1 1 53D2AA11
+P 14500 15300
+F 0 "K2" V 14450 15300 50  0000 C CNN
+F 1 "TR" V 14550 15300 40  0000 C CNN
+F 2 "Connect:PINHEAD1-3" H 14500 15300 60  0001 C CNN
+F 3 "" H 14500 15300 60  0000 C CNN
+	1    14500 15300
+	-1   0    0    1
+$EndComp
+$Comp
+L GND #PWR095
+U 1 1 53D2AA17
+P 15550 15350
+F 0 "#PWR095" H 15550 15350 30  0001 C CNN
+F 1 "GND" H 15550 15280 30  0001 C CNN
+F 2 "" H 15550 15350 60  0000 C CNN
+F 3 "" H 15550 15350 60  0000 C CNN
+	1    15550 15350
+	1    0    0    -1
+$EndComp
+Wire Wire Line
+	14850 15200 15250 15200
+Wire Wire Line
+	14850 15400 15250 15400
+Wire Wire Line
+	14850 15300 15550 15300
+Wire Wire Line
+	15550 15300 15550 15350
+Text Notes 15800 15300 0    79   ~ 0
+to monitor
+Text Notes 15800 13700 0    79   ~ 0
+to driver amplifier
 $EndSCHEMATC

Commit message: added extra power header to control board, added spam to driver amp bottom soldermask layer to pass oshpark check script, added board outlines to agc and tr silkscreen
Parts:
- added K4: VOUT_TR, Connect:PINHEAD1-3, symbol CONN_3
- R28: value DNP -> 0
- R29: value 0 -> DNP
Connections:
- net +5V: now also K4.1 (P1)
- net GND: now also K4.2 (PM)
- net VCC: now also K4.3 (P3)
Other:
- note added: "jumper FWD fault to high.."

Commit message: started on t/r with enclosure, migrated distro to 15v
Connections:
- net +5V: no longer K3.1 (P1)
Other:
- note added: "todo: change resistors for 15V"
Changed lines of the file:
@@
-$EndComp
-$Comp
-L +5V #PWR5
-U 1 1 538507A4
-P 1650 12650
-F 0 "#PWR5" H 1650 12740 20  0001 C CNN
-F 1 "+5V" H 1650 12740 30  0000 C CNN
-F 2 "" H 1650 12650 60  0000 C CNN
-F 3 "" H 1650 12650 60  0000 C CNN
-	1    1650 12650
-	-1   0    0    1
 $EndComp
 $Comp
@@
 Wire Wire Line
 	16300 10150 18300 10150
-Wire Wire Line
-	1450 12200 1650 12200
-Wire Wire Line
-	1650 12200 1650 12650
 Wire Wire Line
 	14800 11850 14800 11950
@@
 Wire Wire Line
 	1550 10850 1450 10850
+Text Notes 17250 8250 0    79   ~ 0
+todo: change resistors for 15V
 $EndSCHEMATC
