File: distro/distro.sch (KiCad schematic (older format))
At the start: 19 parts, among them K1 CONN_3, K2 CONN_3, K3 CONN_3, K4 CONN_3, P4 CONN_2, P5 CONN_2, P6 CONN_2, P7 CONN_2

Commit message: added dfm changes from fab, I think
Parts:
- added D1, D2: LED, LEDs:LED-0805, symbol LED
- added R1: 10k, Resistors_SMD:R_0805, symbol R
- added R2: 100k, Resistors_SMD:R_0805, symbol R
Connections:
- wire segments 43 -> 49
Changed lines of the file:
@@
 LIBS:contrib
 LIBS:valves
-LIBS:kbvw006a0b
+LIBS:sma
+LIBS:npn1b2c3e
+LIBS:mrfe6vp100h
+LIBS:mga-61563
+LIBS:ltc2914
+LIBS:lm2936bm
+LIBS:isl3281e
+LIBS:hmc595
+LIBS:hmc475
+LIBS:ba08cc0wfp
+LIBS:ad9835
+LIBS:75182
+LIBS:7545x
+LIBS:74xx1g14
+LIBS:sclf-25
+LIBS:sky12347
+LIBS:smp1330-005lf
+LIBS:tcm809
+LIBS:7805
 LIBS:mounting_hole
-LIBS:distro-cache
-EELAYER 24 0
+LIBS:swma-2-50dr+
+LIBS:mar-8asm+
+LIBS:ltc1983-5
+LIBS:ldo_78xx
+LIBS:rxfe-cache
+EELAYER 25 0
 EELAYER END
 $Descr A4 11693 8268
@@
 $EndComp
 $Comp
-L +12V #PWR01
+L +12V #PWR1
 U 1 1 5408CCC6
 P 2700 650
-F 0 "#PWR01" H 2700 600 20  0001 C CNN
+F 0 "#PWR1" H 2700 600 20  0001 C CNN
 F 1 "+12V" H 2700 750 30  0000 C CNN
 F 2 "" H 2700 650 60  0000 C CNN
@@
 $EndComp
 $Comp
-L GND #PWR02
+L GND #PWR2
 U 1 1 5408CCD3
 P 2700 1350
-F 0 "#PWR02" H 2700 1350 30  0001 C CNN
+F 0 "#PWR2" H 2700 1350 30  0001 C CNN
 F 1 "GND" H 2700 1280 30  0001 C CNN
 F 2 "" H 2700 1350 60  0000 C CNN
@@
 $EndComp
 $Comp
-L +12V #PWR03
+L +12V #PWR5
 U 1 1 5408CDD1
 P 3050 3850
-F 0 "#PWR03" H 3050 3800 20  0001 C CNN
+F 0 "#PWR5" H 3050 3800 20  0001 C CNN
 F 1 "+12V" H 3050 3950 30  0000 C CNN
 F 2 "" H 3050 3850 60  0000 C CNN
@@
 Fan 0
 $Comp
-L +12V #PWR04
+L +12V #PWR7
 U 1 1 5408CE04
 P 3050 5150
-F 0 "#PWR04" H 3050 5100 20  0001 C CNN
+F 0 "#PWR7" H 3050 5100 20  0001 C CNN
 F 1 "+12V" H 3050 5250 30  0000 C CNN
 F 2 "" H 3050 5150 60  0000 C CNN
@@
 $EndComp
 $Comp
-L GND #PWR05
+L GND #PWR8
 U 1 1 5408CE10
 P 3050 5600
-F 0 "#PWR05" H 3050 5600 30  0001 C CNN
+F 0 "#PWR8" H 3050 5600 30  0001 C CNN
 F 1 "GND" H 3050 5530 30  0001 C CNN
 F 2 "" H 3050 5600 60  0000 C CNN
@@
 $EndComp
 $Comp
-L GND #PWR06
+L GND #PWR22
 U 1 1 5408CFAA
 P 6100 2950
-F 0 "#PWR06" H 6100 2950 30  0001 C CNN
+F 0 "#PWR22" H 6100 2950 30  0001 C CNN
 F 1 "GND" H 6100 2880 30  0001 C CNN
 F 2 "" H 6100 2950 60  0000 C CNN
@@
 $EndComp
 $Comp
-L GND #PWR07
+L GND #PWR20
 U 1 1 5408CFC7
 P 6100 2200
-F 0 "#PWR07" H 6100 2200 30  0001 C CNN
+F 0 "#PWR20" H 6100 2200 30  0001 C CNN
 F 1 "GND" H 6100 2130 30  0001 C CNN
 F 2 "" H 6100 2200 60  0000 C CNN
@@
 Driver amp power
 $Comp
-L GND #PWR08
+L GND #PWR4
 U 1 1 5408CFEC
 P 3050 3350
-F 0 "#PWR08" H 3050 3350 30  0001 C CNN
+F 0 "#PWR4" H 3050 3350 30  0001 C CNN
 F 1 "GND" H 3050 3280 30  0001 C CNN
 F 2 "" H 3050 3350 60  0000 C CNN
@@
 NoConn ~ 2850 3350
 $Comp
-L +12V #PWR09
+L +12V #PWR3
 U 1 1 5408D027
 P 3050 2950
-F 0 "#PWR09" H 3050 2900 20  0001 C CNN
+F 0 "#PWR3" H 3050 2900 20  0001 C CNN
 F 1 "+12V" H 3050 3050 30  0000 C CNN
 F 2 "" H 3050 2950 60  0000 C CNN
@@
 Control power
 $Comp
-L VCC #PWR010
+L VCC #PWR19
 U 1 1 5408D094
 P 6100 1700
-F 0 "#PWR010" H 6100 1800 30  0001 C CNN
+F 0 "#PWR19" H 6100 1800 30  0001 C CNN
 F 1 "VCC" H 6100 1800 30  0000 C CNN
 F 2 "" H 6100 1700 60  0000 C CNN
@@
 $EndComp
 $Comp
-L VCC #PWR011
+L VCC #PWR21
 U 1 1 5408D0D1
 P 6100 2450
-F 0 "#PWR011" H 6100 2550 30  0001 C CNN
+F 0 "#PWR21" H 6100 2550 30  0001 C CNN
 F 1 "VCC" H 6100 2550 30  0000 C CNN
 F 2 "" H 6100 2450 60  0000 C CNN
@@
 $EndComp
 $Comp
-L GND #PWR012
+L GND #PWR24
 U 1 1 5408D56B
 P 6100 3750
-F 0 "#PWR012" H 6100 3750 30  0001 C CNN
+F 0 "#PWR24" H 6100 3750 30  0001 C CNN
 F 1 "GND" H 6100 3680 30  0001 C CNN
 F 2 "" H 6100 3750 60  0000 C CNN
@@
 50V in
 $Comp
-L VCC #PWR013
+L VCC #PWR23
 U 1 1 5408D576
 P 6100 3250
-F 0 "#PWR013" H 6100 3350 30  0001 C CNN
+F 0 "#PWR23" H 6100 3350 30  0001 C CNN
 F 1 "VCC" H 6100 3350 30  0000 C CNN
 F 2 "" H 6100 3250 60  0000 C CNN
@@
 $EndComp
 $Comp
-L GND #PWR014
+L GND #PWR16
 U 1 1 5408D709
 P 5650 1400
-F 0 "#PWR014" H 5650 1400 30  0001 C CNN
+F 0 "#PWR16" H 5650 1400 30  0001 C CNN
 F 1 "GND" H 5650 1330 30  0001 C CNN
 F 2 "" H 5650 1400 60  0000 C CNN
@@
 $EndComp
 $Comp
-L VCC #PWR015
+L VCC #PWR15
 U 1 1 5408D711
 P 5650 700
-F 0 "#PWR015" H 5650 800 30  0001 C CNN
+F 0 "#PWR15" H 5650 800 30  0001 C CNN
 F 1 "VCC" H 5650 800 30  0000 C CNN
 F 2 "" H 5650 700 60  0000 C CNN
@@
 $EndComp
 $Comp
-L VCC #PWR016
+L VCC #PWR25
 U 1 1 5408E181
 P 6700 700
-F 0 "#PWR016" H 6700 800 30  0001 C CNN
+F 0 "#PWR25" H 6700 800 30  0001 C CNN
 F 1 "VCC" H 6700 800 30  0000 C CNN
 F 2 "" H 6700 700 60  0000 C CNN
@@
 $EndComp
 $Comp
-L GND #PWR017
+L GND #PWR26
 U 1 1 5408E18C
 P 6700 1400
-F 0 "#PWR017" H 6700 1400 30  0001 C CNN
+F 0 "#PWR26" H 6700 1400 30  0001 C CNN
 F 1 "GND" H 6700 1330 30  0001 C CNN
 F 2 "" H 6700 1400 60  0000 C CNN
@@
 $EndComp
 $Comp
-L GND #PWR018
+L GND #PWR28
 U 1 1 5408E197
 P 6950 1400
-F 0 "#PWR018" H 6950 1400 30  0001 C CNN
+F 0 "#PWR28" H 6950 1400 30  0001 C CNN
 F 1 "GND" H 6950 1330 30  0001 C CNN
 F 2 "" H 6950 1400 60  0000 C CNN
@@
 $EndComp
 $Comp
-L +12V #PWR019
+L +12V #PWR27
 U 1 1 5408E1B1
 P 6950 700
-F 0 "#PWR019" H 6950 650 20  0001 C CNN
+F 0 "#PWR27" H 6950 650 20  0001 C CNN
 F 1 "+12V" H 6950 800 30  0000 C CNN
 F 2 "" H 6950 700 60  0000 C CNN
@@
 $EndComp
 $Comp
-L +12V #PWR020
+L +12V #PWR9
 U 1 1 5408F29B
 P 3050 5850
-F 0 "#PWR020" H 3050 5800 20  0001 C CNN
+F 0 "#PWR9" H 3050 5800 20  0001 C CNN
 F 1 "+12V" H 3050 5950 30  0000 C CNN
 F 2 "" H 3050 5850 60  0000 C CNN
@@
 $EndComp
 $Comp
-L GND #PWR021
+L GND #PWR10
 U 1 1 5408F2A7
 P 3050 6300
-F 0 "#PWR021" H 3050 6300 30  0001 C CNN
+F 0 "#PWR10" H 3050 6300 30  0001 C CNN
 F 1 "GND" H 3050 6230 30  0001 C CNN
 F 2 "" H 3050 6300 60  0000 C CNN
@@
 15V MON
 $Comp
-L +12V #PWR022
+L +12V #PWR11
 U 1 1 5417210E
 P 3050 6600
-F 0 "#PWR022" H 3050 6550 20  0001 C CNN
+F 0 "#PWR11" H 3050 6550 20  0001 C CNN
 F 1 "+12V" H 3050 6700 30  0000 C CNN
 F 2 "" H 3050 6600 60  0000 C CNN
@@
 $EndComp
 $Comp
-L GND #PWR023
+L GND #PWR12
 U 1 1 5417211A
 P 3050 7050
-F 0 "#PWR023" H 3050 7050 30  0001 C CNN
+F 0 "#PWR12" H 3050 7050 30  0001 C CNN
 F 1 "GND" H 3050 6980 30  0001 C CNN
 F 2 "" H 3050 7050 60  0000 C CNN
@@
 	5650 700  5650 850
 Wire Wire Line
-	6950 700  6950 800
-Wire Wire Line
-	6700 700  6700 800
-Wire Wire Line
-	6700 1200 6700 1400
-Wire Wire Line
-	6950 1200 6950 1400
+	6950 700  6950 850
+Wire Wire Line
+	6700 700  6700 850
+Wire Wire Line
+	6700 1150 6700 1400
+Wire Wire Line
+	6950 1150 6950 1400
 Wire Wire Line
 	2850 5950 3050 5950
@@
 	2850 4150 3050 4150
 $Comp
-L GND #PWR024
+L GND #PWR6
 U 1 1 5408CDDD
 P 3050 4300
-F 0 "#PWR024" H 3050 4300 30  0001 C CNN
+F 0 "#PWR6" H 3050 4300 30  0001 C CNN
 F 1 "GND" H 3050 4230 30  0001 C CNN
 F 2 "" H 3050 4300 60  0000 C CNN
@@
 	2850 6050 3050 6050
 Connection ~ 3050 6150
+$Comp
+L R R1
+U 1 1 55359326
+P 5550 4800
+F 0 "R1" V 5630 4800 50  0000 C CNN
+F 1 "10k" V 5550 4800 50  0000 C CNN
+F 2 "Resistors_SMD:R_0805" V 5480 4800 30  0001 C CNN
+F 3 "" H 5550 4800 30  0000 C CNN
+	1    5550 4800
+	1    0    0    -1
+$EndComp
+$Comp
+L R R2
+U 1 1 55359379
+P 5800 4800
+F 0 "R2" V 5880 4800 50  0000 C CNN
+F 1 "100k" V 5800 4800 50  0000 C CNN
+F 2 "Resistors_SMD:R_0805" V 5730 4800 30  0001 C CNN
+F 3 "" H 5800 4800 30  0000 C CNN
+	1    5800 4800
+	1    0    0    -1
+$EndComp
+$Comp
+L LED D1
+U 1 1 553593F5
+P 5550 5250
+F 0 "D1" H 5550 5350 50  0000 C CNN
+F 1 "LED" H 5550 5150 50  0000 C CNN
+F 2 "LEDs:LED-0805" H 5550 5250 60  0001 C CNN
+F 3 "" H 5550 5250 60  0000 C CNN
+	1    5550 5250
+	0    1    1    0
+$EndComp
+$Comp
+L LED D2
+U 1 1 553594AE
+P 5800 5250
+F 0 "D2" H 5800 5350 50  0000 C CNN
+F 1 "LED" H 5800 5150 50  0000 C CNN
+F 2 "LEDs:LED-0805" H 5800 5250 60  0001 C CNN
+F 3 "" H 5800 5250 60  0000 C CNN
+	1    5800 5250
+	0    1    1    0
+$EndComp
+$Comp
+L GND #PWR18
+U 1 1 553594FC
+P 5800 5500
+F 0 "#PWR18" H 5800 5500 30  0001 C CNN
+F 1 "GND" H 5800 5430 30  0001 C CNN
+F 2 "" H 5800 5500 60  0000 C CNN
+F 3 "" H 5800 5500 60  0000 C CNN
+	1    5800 5500
+	1    0    0    -1
+$EndComp
+$Comp
+L VCC #PWR17
+U 1 1 5535954C
+P 5800 4600
+F 0 "#PWR17" H 5800 4700 30  0001 C CNN
+F 1 "VCC" H 5800 4700 30  0000 C CNN
+F 2 "" H 5800 4600 60  0000 C CNN
+F 3 "" H 5800 4600 60  0000 C CNN
+	1    5800 4600
+	1    0    0    -1
+$EndComp
+$Comp
+L +12V #PWR13
+U 1 1 55359BB8
+P 5550 4600
+F 0 "#PWR13" H 5550 4550 20  0001 C CNN
+F 1 "+12V" H 5550 4700 30  0000 C CNN
+F 2 "" H 5550 4600 60  0000 C CNN
+F 3 "" H 5550 4600 60  0000 C CNN
+	1    5550 4600
+	1    0    0    -1
+$EndComp
+$Comp
+L GND #PWR14
+U 1 1 55359BF1
+P 5550 5500
+F 0 "#PWR14" H 5550 5500 30  0001 C CNN
+F 1 "GND" H 5550 5430 30  0001 C CNN
+F 2 "" H 5550 5500 60  0000 C CNN
+F 3 "" H 5550 5500 60  0000 C CNN
+	1    5550 5500
+	1    0    0    -1
+$EndComp
+Wire Wire Line
+	5800 4600 5800 4650
+Wire Wire Line
+	5550 4600 5550 4650
+Wire Wire Line
+	5550 4950 5550 5050
+Wire Wire Line
+	5550 5450 5550 5500
+Wire Wire Line
+	5800 5450 5800 5500
+Wire Wire Line
+	5800 4950 5800 5050
 $EndSCHEMATC
