File: rxfe/rxfe.kicad_pcb (KiCad board)
At the start: 2 copper layers, 129.5 x 46.2 mm, 83 parts, among them J1 SMA, J2 SMA, J3 4610X-AP1-103LF, J4 SMA, K1 CONN_3, P1 CONN_8X2, U1 SKY12347, U10 SMP1330-005LF, U11 LTC1983-5, U12 SMP1330-005LF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

Commit message: DFM changes after last protoype rev
Routing:
- net GND: track 264.2 -> 262.9 mm, vias 121 -> 119
Other:
- rule via_min_drill: 0.508 -> 0.33
- rule via_min_size: 0.889 -> 0.6
- board text added: "c"

Commit message: finalized driveramp, rxfe, and control for macrofab
Parts:
- removed C19, C2, C31, C32: 100 nF, SMD_Packages:SMD-0805
- added R12: 1k, Resistors_SMD:R_0805, F.Cu at (111.8, 103.4)
- added R7: 1k, Resistors_SMD:R_0805, F.Cu at (109.2, 103.4)
- C1, C29, C5: value 100 nF -> 22 nF; footprint SMD_Packages:SMD-0805 -> Capacitors_SMD:C_0805
- C10, C11, C12, C13, C14, C15, C16, C17, C18, C20, C21, C22, C23, C24, C25, C26, C27, C28, C3, C30, C36, C37, C4, C9: footprint SMD_Packages:SMD-0805 -> Capacitors_SMD:C_0805
- C6: footprint SMD_Packages:SMD-1210 -> SMD_Packages:SMD-1210_Pol
- C7, C8: footprint SMD_Packages:SMD-1210 -> Capacitors_SMD:C_1210
- D1: footprint SMD_Packages:SMD-0805 -> LEDs:LED-0805
- L1, L2, L3: footprint SMD_Packages:SMD-1210 -> Resistors_SMD:R_1210
- L4, L6, L7: value 10 uH -> 3.9uH; footprint SMD_Packages:SMD-0805 -> Resistors_SMD:R_1210
- L5: value 10 uH -> 3.9uH; footprint SMD_Packages:SMD-1210 -> Resistors_SMD:R_1210
- R1, R2, R3, R4, R5, R6, R8: footprint SMD_Packages:SMD-0805 -> Resistors_SMD:R_0805
- R10, R11: value 309 -> 93.1; footprint SMD_Packages:SMD-1210 -> Resistors_SMD:R_1210
- R9: value 309 -> 1k; footprint SMD_Packages:SMD-1210 -> Resistors_SMD:R_0805
- U8: value MASWSS0179' -> MASWSS0179
- moved R9 3.07 mm to (106.7, 103.4)
- moved C24 2.29 mm to (171.2, 100.6)
- moved C18 1.00 mm to (103.1, 103.5), turned to 0 degrees
- moved L4 0.81 mm to (110.2, 99.6)
- moved L7 0.59 mm to (170.2, 103.6)
- moved R11 0.34 mm to (168.1, 107.4)
Connections:
- net VCC renamed +5V
- U1 pad 15: (no net) -> Net-(U1-Pad15)
- U2 pad 10: (no net) -> Net-(U2-Pad10)
- U2 pad 6: (no net) -> Net-(U2-Pad6)
Routing:
- net /T/R: track 88.1 -> 93.9 mm
- net Net-(L4-Pad2): track 2.57 -> 8.12 mm
- net VDD: track 150.0 -> 155.5 mm
- net (no net): track 0.00 -> 4.17 mm, vias 0 -> 3
- net GND: track 262.9 -> 260.8 mm, vias 119 -> 126
- net +5V: track 184.4 -> 183.1 mm
- net Net-(C23-Pad2): track 5.20 -> 5.96 mm

Commit message: added dfm changes from fab, I think
Parts:
- added C19: 22 nF, Capacitors_SMD:C_0805, F.Cu at (162.6, 98.6)
- added C2: 22 nF, Capacitors_SMD:C_0805, F.Cu at (197.4, 96.3)
- added C31: 22 nF, Capacitors_SMD:C_0805, F.Cu at (207.3, 97.3)
- added C32: 22 nF, Capacitors_SMD:C_0805, F.Cu at (170.9, 98.8)
- C1, C18, C20, C21, C27, C28, C29, C4, C5: value 22 nF -> 100 nF
- moved C24 2.51 mm to (173.0, 102.4), turned to 270 degrees
- moved FID3 1.02 mm to (205.0, 88.1)
Connections:
- net +5V renamed VCC
- U4 pad 2: GND -> Net-(C2-Pad2)
- U5 pad 2: GND -> Net-(C19-Pad2)
- U8 pad 2: GND -> Net-(C31-Pad1)
- U9 pad 2: GND -> Net-(C32-Pad1)
Routing:
- net VDD: track 155.5 -> 151.3 mm
- net (no net): track 4.17 -> 0.00 mm, vias 3 -> 0
- net Net-(C32-Pad1): track 0.00 -> 2.08 mm
- net Net-(C24-Pad2): track 4.69 -> 6.74 mm
- net Net-(C19-Pad2): track 0.00 -> 1.93 mm
- net Net-(C15-Pad2): track 9.88 -> 11.8 mm
- net Net-(C17-Pad2): track 9.35 -> 11.2 mm
- net Net-(C2-Pad2): track 0.00 -> 1.70 mm
- net Net-(C31-Pad1): track 0.00 -> 1.67 mm
- net GND: track 260.8 -> 259.8 mm
Other:
- board text removed: "c"
