File: rxfe/rxfe.sch (KiCad schematic (older format))
At the start: 81 parts, among them J1 SMA, J2 SMA, J3 4610X-AP1-103LF, J4 SMA, K1 CONN_3, P1 CONN_8X2, U1 SKY12347, U10 SMP1330-005LF, U11 LTC1983-5, U12 SMP1330-005LF, U13 LDO_78XX, U14 TCM809, U15 GALI-84+, U16 GALI-84+, U2 74HC04, U3 SCLF-25, U4 MASWSS0179, U5 MASWSS0179, U6 MAR-8ASM+, U7 SWMA-2-50DR+, U8 MASWSS0179, U9 MASWSS0179

Commit message: finalized driveramp, rxfe, and control for macrofab
Parts:
- C1, C10, C11, C12, C13, C14, C15, C16, C17, C18, C20, C21, C22, C23, C24, C25, C26, C27, C28, C29, C3, C30, C36, C37, C4, C5, C9: footprint SMD_Packages:SMD-0805 -> Capacitors_SMD:C_0805
- C7, C8: footprint SMD_Packages:SMD-1206_Pol -> Capacitors_SMD:C_1210
- D1: footprint SMD_Packages:SMD-0805 -> LEDs:LED-0805
- L1, L2, L3, L5, R10, R11: footprint SMD_Packages:SMD-1210 -> Resistors_SMD:R_1210
- L4, L6, L7: footprint SMD_Packages:SMD-0805 -> Resistors_SMD:R_1210
- R1, R12, R2, R3, R4, R5, R6, R7, R8: footprint SMD_Packages:SMD-0805 -> Resistors_SMD:R_0805
- R9: footprint SMD_Packages:SMD-1210 -> Resistors_SMD:R_0805
Connections:
- net labels removed: VCC
- wire segments 258 -> 260

Commit message: added dfm changes from fab, I think
Parts:
- added C19, C2, C31, C32: 22 nF, Capacitors_SMD:C_0805, symbol C
- C1, C18, C20, C21, C27, C28, C29, C4, C5: value 22 nF -> 100 nF
- U4, U5, U8, U9: value MASWSS0179 -> MASW-007935-TR3000; MFG PN MASWSS0179TR-3000 -> MASW-007935-TR3000
Connections:
- net GND: now also C19.1, C2.1, C31.2, C32.2; no longer U4.2 (GND), U5.2 (GND), U8.2 (GND), U9.2 (GND)
- new net: C19.2, U5.2 (GND)
- new net: C32.1, U9.2 (GND)
- new net: C2.2, U4.2 (GND)
- new net: C31.1, U8.2 (GND)
Other:
- moved on the sheet: C11, C13, C23, C24

Commit message: added some notes/errata to the transmitter schematics
Parts:
- D1: symbol LED -> LED-RESCUE-rxfe
- U3: symbol SCLF-25 -> SCLF-25-RESCUE-rxfe
Other:
- note added: "A402G\n"
- note added: "TODO: ADD IO ISOLATION"
- note added: "TODO: replace all connectors with through hole!"
- note added: "check power dissipation\n"
- note added: "replace with HMC849?"
- note added: "replace with SOT89? replace with TI chip?"
- note added: "replace with TI chip?"
- note added: "switch to stocked part (see mcm rxfe)"
Changed lines of the file:
@@
 EESchema Schematic File Version 2
+LIBS:rxfe-rescue
 LIBS:power
 LIBS:device
@@
 LIBS:memory
 LIBS:xilinx
-LIBS:special
 LIBS:microcontrollers
 LIBS:dsp
@@
 $EndComp
 $Comp
-L SCLF-25 U3
+L SCLF-25-RESCUE-rxfe U3
 U 1 1 53B49227
 P 13050 3950
@@
 AMP1CTL
 $Comp
-L LED D1
+L LED-RESCUE-rxfe D1
 U 1 1 53B876A5
 P 12000 14200
@@
 Wire Wire Line
 	9600 12050 9600 11600
+Text Notes 6300 2950 0    118  ~ 24
+replace with HMC849?
+Text Notes 2900 2700 0    60   ~ 0
+replace with SOT89? replace with TI chip?
+Text Notes 10050 7400 0    60   ~ 0
+A402G\n
+Text Notes 10000 7300 0    118  ~ 24
+replace with TI chip?
+Text Notes 9700 11200 0    60   ~ 0
+replace with TI chip?
+Text Notes 9650 13950 0    60   ~ 0
+check power dissipation\n
+Text Notes 3050 11100 0    118  ~ 24
+switch to stocked part (see mcm rxfe)
+Text Notes 10650 1900 0    118  ~ 24
+TODO: ADD IO ISOLATION
+Text Notes 10700 2100 0    118  ~ 24
+TODO: replace all connectors with through hole!
 $EndSCHEMATC
