File: usrp_dio/usrp_dio.sch (KiCad schematic (older format))
At the start: 8 parts, among them P1 CONN_01X15, P2 CONN_02X08, P3 CONN_02X08, P4 CONN_02X08, P5 CONN_02X08, U1 74HC595

Commit message: committing modified files, I forget.., probably dfm
Parts:
- P1: DIST_PN AE10974-ND -> AE10978-ND; MAN_PN ADS15A-KG-TASB3-R -> A-DS-15-LL/Z
Changed lines of the file:
@@
 F 3 "" H 1950 3550 60  0000 C CNN
 F 4 "Assmann WSW Components" H 1950 3550 60  0001 C CNN "MAN_NAME"
-F 5 "ADS15A-KG-TASB3-R" H 1950 3550 60  0001 C CNN "MAN_PN"
+F 5 "A-DS-15-LL/Z" H 1950 3550 60  0001 C CNN "MAN_PN"
 F 6 "DigiKey" H 1950 3550 60  0001 C CNN "DIST_NAME"
-F 7 "AE10974-ND" H 1950 3550 60  0001 C CNN "DIST_PN"
+F 7 "AE10978-ND" H 1950 3550 60  0001 C CNN "DIST_PN"
 	1    1950 3550
 	-1   0    0    1

Commit message: added dfm changes from fab, I think
Parts:
- added J?: SMA, symbol SMA
- added P? (x2): CONN_01X02, symbol CONN_01X02
- added R?: R, symbol R
Connections:
- net +3V3: now also U1.10 (SRCLR)
- net D0: now also R?.1; no longer U1.13 (G)
- net D1: now also P?.1 (P1); no longer U1.12 (RCLK)
- net D2: now also P?.1 (P1); no longer U1.10 (SRCLR)
- net D3: now also U1.12 (RCLK)
- net GND: now also U1.13 (G), J?.2 (GND), J?.3 (GND), J?.4 (GND), J?.5 (GND), P?.2 (P2), P?.2 (P2)
- new net: J?.1 (RF), R?.2
Other:
- note added: "force D8/D9 as differential in hardware\nsee MAX3293 or ISL3295EFHZ"
- note added: "mates with 89116-0101"

Commit message: updated usrp dio layout to send more gpio lines to agc boards
Parts:
- added D?: LED, symbol LED
- added R?: R, Resistors_SMD:R_0805, symbol R
- J1: renamed from J?; footprint (none) -> local:SMA_5-1814832-1
- P1: footprint Connect:DB15M_CI -> sdtransmitter:182-015-113R531_dsub15
- P6, P7: renamed from P?; footprint (none) -> Connect:PINHEAD1-2
- R1: renamed from R?; footprint (none) -> Resistors_SMD:R_0805
Connections:
- net +3V3: now also D?.1 (A)
- net D0: now also P6.1 (P1); no longer R1.1
- net D2: now also R1.1; no longer P6.1 (P1)
- net D3: now also U1.14 (SER); no longer U1.11 (SRCLK), U1.12 (RCLK)
- net D4: now also U1.11 (SRCLK), U1.12 (RCLK); no longer U1.14 (SER)
- net GND: now also R?.1
- new net: D?.2 (K), R?.2
Other:
- note added: "output enable, active low"
- note added: "rclk and sclk, shift and storage register clocks"
- note added: "serial data in"
- note added: "srclr is active low master reset"
Changed lines of the file:
@@
 F 0 "P1" H 1950 4350 50  0000 C CNN
 F 1 "CONN_01X15" V 2050 3550 50  0000 C CNN
-F 2 "Connect:DB15M_CI" H 1950 3550 60  0001 C CNN
+F 2 "sdtransmitter:182-015-113R531_dsub15" H 1950 3550 60  0001 C CNN
 F 3 "" H 1950 3550 60  0000 C CNN
 F 4 "Assmann WSW Components" H 1950 3550 60  0001 C CNN "MAN_NAME"
@@
 $EndComp
 $Comp
-L +3.3V #PWR3
+L +3.3V #PWR01
 U 1 1 5511FEDD
 P 2300 4250
-F 0 "#PWR3" H 2300 4100 50  0001 C CNN
+F 0 "#PWR01" H 2300 4100 50  0001 C CNN
 F 1 "+3.3V" V 2400 4250 50  0000 C CNN
 F 2 "" H 2300 4250 60  0000 C CNN
@@
 $EndComp
 $Comp
-L GND #PWR1
+L GND #PWR02
 U 1 1 5511FF0B
 P 2300 2850
-F 0 "#PWR1" H 2300 2600 50  0001 C CNN
+F 0 "#PWR02" H 2300 2600 50  0001 C CNN
 F 1 "GND" V 2350 2650 50  0000 C CNN
 F 2 "" H 2300 2850 60  0000 C CNN
@@
 $EndComp
 $Comp
-L GND #PWR2
+L GND #PWR03
 U 1 1 5511FF20
 P 2300 2950
-F 0 "#PWR2" H 2300 2700 50  0001 C CNN
+F 0 "#PWR03" H 2300 2700 50  0001 C CNN
 F 1 "GND" V 2350 2750 50  0000 C CNN
 F 2 "" H 2300 2950 60  0000 C CNN
@@
 $EndComp
 $Comp
-L GND #PWR7
+L GND #PWR04
 U 1 1 5512016B
 P 5950 2050
-F 0 "#PWR7" H 5950 1800 50  0001 C CNN
+F 0 "#PWR04" H 5950 1800 50  0001 C CNN
 F 1 "GND" H 5950 1900 50  0000 C CNN
 F 2 "" H 5950 2050 60  0000 C CNN
@@
 $EndComp
 $Comp
-L GND #PWR6
+L GND #PWR05
 U 1 1 55120573
 P 5600 4500
-F 0 "#PWR6" H 5600 4250 50  0001 C CNN
+F 0 "#PWR05" H 5600 4250 50  0001 C CNN
 F 1 "GND" H 5600 4350 50  0000 C CNN
 F 2 "" H 5600 4500 60  0000 C CNN
@@
 $EndComp
 $Comp
-L GND #PWR5
+L GND #PWR06
 U 1 1 5512077B
 P 4450 4500
-F 0 "#PWR5" H 4450 4250 50  0001 C CNN
+F 0 "#PWR06" H 4450 4250 50  0001 C CNN
 F 1 "GND" H 4450 4350 50  0000 C CNN
 F 2 "" H 4450 4500 60  0000 C CNN
@@
 $EndComp
 $Comp
-L GND #PWR10
+L GND #PWR07
 U 1 1 55120949
 P 7100 2050
-F 0 "#PWR10" H 7100 1800 50  0001 C CNN
+F 0 "#PWR07" H 7100 1800 50  0001 C CNN
 F 1 "GND" H 7100 1900 50  0000 C CNN
 F 2 "" H 7100 2050 60  0000 C CNN
@@
 	1    0    0    -1
 $EndComp
-Text Label 8400 5650 0    60   ~ 0
+Text Label 8350 3950 2    60   ~ 0
 D0
 Text Label 8350 4450 2    60   ~ 0
 D1
-Text Label 8350 3950 2    60   ~ 0
+Text Label 8400 5650 0    60   ~ 0
 D2
-Text Label 6450 2500 0    60   ~ 0
+Text Label 5800 2700 2    60   ~ 0
 D4
-Text Label 5800 2700 0    60   ~ 0
+Text Label 6450 2500 2    60   ~ 0
 D3
 Text Label 4750 3900 0    60   ~ 0
@@
 $EndComp
 $Comp
-L VCC #PWR4
+L VCC #PWR08
 U 1 1 55135D0F
 P 2350 4500
-F 0 "#PWR4" H 2350 4350 50  0001 C CNN
+F 0 "#PWR08" H 2350 4350 50  0001 C CNN
 F 1 "VCC" H 2350 4650 50  0000 C CNN
 F 2 "" H 2350 4500 60  0000 C CNN
@@
 $EndComp
 $Comp
-L VCC #PWR8
+L VCC #PWR09
 U 1 1 55135DBF
 P 7050 4100
-F 0 "#PWR8" H 7050 3950 50  0001 C CNN
+F 0 "#PWR09" H 7050 3950 50  0001 C CNN
 F 1 "VCC" H 7050 4250 50  0000 C CNN
 F 2 "" H 7050 4100 60  0000 C CNN
@@
 $EndComp
 $Comp
-L GND #PWR9
+L GND #PWR010
 U 1 1 55135E77
 P 7050 4600
-F 0 "#PWR9" H 7050 4350 50  0001 C CNN
+F 0 "#PWR010" H 7050 4350 50  0001 C CNN
 F 1 "GND" H 7050 4450 50  0000 C CNN
 F 2 "" H 7050 4600 60  0000 C CNN
@@
 NoConn ~ 5000 3700
 $Comp
-L VCC #PWR11
+L VCC #PWR011
 U 1 1 55139310
 P 7500 4100
-F 0 "#PWR11" H 7500 3950 50  0001 C CNN
+F 0 "#PWR011" H 7500 3950 50  0001 C CNN
 F 1 "VCC" H 7500 4250 50  0000 C CNN
 F 2 "" H 7500 4100 60  0000 C CNN
@@
 $EndComp
 $Comp
-L GND #PWR12
+L GND #PWR012
 U 1 1 5513931C
 P 7500 4600
-F 0 "#PWR12" H 7500 4350 50  0001 C CNN
+F 0 "#PWR012" H 7500 4350 50  0001 C CNN
 F 1 "GND" H 7500 4450 50  0000 C CNN
 F 2 "" H 7500 4600 60  0000 C CNN
@@
 mates with 89116-0101
 $Comp
-L VCC #PWR?
+L VCC #PWR013
 U 1 1 5547CA1B
 P 6450 2800
-F 0 "#PWR?" H 6450 2650 50  0001 C CNN
+F 0 "#PWR013" H 6450 2650 50  0001 C CNN
 F 1 "VCC" H 6450 2950 50  0000 C CNN
 F 2 "" H 6450 2800 60  0000 C CNN
@@
 $EndComp
 $Comp
-L GND #PWR?
+L GND #PWR014
 U 1 1 5547CB7F
 P 6400 3150
-F 0 "#PWR?" H 6400 2900 50  0001 C CNN
+F 0 "#PWR014" H 6400 2900 50  0001 C CNN
 F 1 "GND" H 6400 3000 50  0000 C CNN
 F 2 "" H 6400 3150 60  0000 C CNN
@@
 $EndComp
 $Comp
-L SMA J?
+L SMA J1
 U 1 1 554804CD
 P 7300 5550
-F 0 "J?" H 7300 5800 60  0000 C CNN
+F 0 "J1" H 7300 5800 60  0000 C CNN
 F 1 "SMA" H 7300 5900 60  0000 C CNN
-F 2 "" H 7300 5800 60  0000 C CNN
+F 2 "local:SMA_5-1814832-1" H 7300 5800 60  0001 C CNN
 F 3 "" H 7300 5800 60  0000 C CNN
 	1    7300 5550
@@
 $EndComp
 $Comp
-L GND #PWR?
+L GND #PWR015
 U 1 1 55480DCB
 P 6600 5900
-F 0 "#PWR?" H 6600 5650 50  0001 C CNN
+F 0 "#PWR015" H 6600 5650 50  0001 C CNN
 F 1 "GND" H 6600 5750 50  0000 C CNN
 F 2 "" H 6600 5900 60  0000 C CNN
@@
 $EndComp
 $Comp
-L R R?
+L R R1
 U 1 1 554810B8
 P 8000 5650
-F 0 "R?" V 8080 5650 50  0000 C CNN
+F 0 "R1" V 8080 5650 50  0000 C CNN
 F 1 "R" V 8000 5650 50  0000 C CNN
-F 2 "" V 7930 5650 30  0000 C CNN
+F 2 "Resistors_SMD:R_0805" V 7930 5650 30  0001 C CNN
 F 3 "" H 8000 5650 30  0000 C CNN
 	1    8000 5650
@@
 	8400 5650 8150 5650
 $Comp
-L CONN_01X02 P?
+L CONN_01X02 P7
 U 1 1 55482BE4
 P 8650 4500
-F 0 "P?" H 8650 4650 50  0000 C CNN
+F 0 "P7" H 8650 4650 50  0000 C CNN
 F 1 "CONN_01X02" V 8750 4500 50  0000 C CNN
-F 2 "" H 8650 4500 60  0000 C CNN
+F 2 "Connect:PINHEAD1-2" H 8650 4500 60  0001 C CNN
 F 3 "" H 8650 4500 60  0000 C CNN
 	1    8650 4500
@@
 $EndComp
 $Comp
-L CONN_01X02 P?
+L CONN_01X02 P6
 U 1 1 55482C4D
 P 8650 4000
-F 0 "P?" H 8650 4150 50  0000 C CNN
+F 0 "P6" H 8650 4150 50  0000 C CNN
 F 1 "CONN_01X02" V 8750 4000 50  0000 C CNN
-F 2 "" H 8650 4000 60  0000 C CNN
+F 2 "Connect:PINHEAD1-2" H 8650 4000 60  0001 C CNN
 F 3 "" H 8650 4000 60  0000 C CNN
 	1    8650 4000
@@
 	8350 4450 8450 4450
 $Comp
-L GND #PWR?
+L GND #PWR016
 U 1 1 55482E83
 P 8350 4050
-F 0 "#PWR?" H 8350 3800 50  0001 C CNN
+F 0 "#PWR016" H 8350 3800 50  0001 C CNN
 F 1 "GND" H 8350 3900 50  0000 C CNN
 F 2 "" H 8350 4050 60  0000 C CNN
@@
 	8450 4050 8350 4050
 $Comp
-L GND #PWR?
+L GND #PWR017
 U 1 1 55482FFD
 P 8350 4550
-F 0 "#PWR?" H 8350 4300 50  0001 C CNN
+F 0 "#PWR017" H 8350 4300 50  0001 C CNN
 F 1 "GND" H 8350 4400 50  0000 C CNN
 F 2 "" H 8350 4550 60  0000 C CNN
@@
 Text Notes 3500 5000 0    60   ~ 0
 force D8/D9 as differential in hardware\nsee MAX3293 or ISL3295EFHZ
+Text Notes 5700 3400 0    60   ~ 0
+output enable, active low
+Text Notes 3700 2850 0    60   ~ 0
+rclk and sclk, shift and storage register clocks
+Text Notes 3700 2950 0    60   ~ 0
+srclr is active low master reset
+Text Notes 5750 2500 0    60   ~ 0
+serial data in
+$Comp
+L LED D?
+U 1 1 559330F0
+P 6600 4350
+F 0 "D?" H 6600 4450 50  0000 C CNN
+F 1 "LED" H 6600 4250 50  0000 C CNN
+F 2 "" H 6600 4350 60  0000 C CNN
+F 3 "" H 6600 4350 60  0000 C CNN
+	1    6600 4350
+	0    1    1    0
+$EndComp
+$Comp
+L VCC #PWR?
+U 1 1 559331B7
+P 6600 4050
+F 0 "#PWR?" H 6600 3900 50  0001 C CNN
+F 1 "VCC" H 6600 4200 50  0000 C CNN
+F 2 "" H 6600 4050 60  0000 C CNN
+F 3 "" H 6600 4050 60  0000 C CNN
+	1    6600 4050
+	1    0    0    -1
+$EndComp
+$Comp
+L R R?
+U 1 1 559331E9
+P 6600 4800
+F 0 "R?" V 6680 4800 50  0000 C CNN
+F 1 "R" V 6600 4800 50  0000 C CNN
+F 2 "Resistors_SMD:R_0805" V 6530 4800 30  0001 C CNN
+F 3 "" H 6600 4800 30  0000 C CNN
+	1    6600 4800
+	-1   0    0    1
+$EndComp
+Wire Wire Line
+	6600 4050 6600 4150
+Wire Wire Line
+	6600 4550 6600 4650
+$Comp
+L GND #PWR?
+U 1 1 559333A4
+P 6600 5000
+F 0 "#PWR?" H 6600 4750 50  0001 C CNN
+F 1 "GND" H 6600 4850 50  0000 C CNN
+F 2 "" H 6600 5000 60  0000 C CNN
+F 3 "" H 6600 5000 60  0000 C CNN
+	1    6600 5000
+	1    0    0    -1
+$EndComp
+Wire Wire Line
+	6600 5000 6600 4950
 $EndSCHEMATC

Commit message: added missing dxf files..
Parts:
- D1: renamed from D?; footprint (none) -> LEDs:LED-0805
- gave numbers to parts that had none: 1
Changed lines of the file:
@@
 serial data in
 $Comp
-L LED D?
+L LED D1
 U 1 1 559330F0
 P 6600 4350
-F 0 "D?" H 6600 4450 50  0000 C CNN
+F 0 "D1" H 6600 4450 50  0000 C CNN
 F 1 "LED" H 6600 4250 50  0000 C CNN
-F 2 "" H 6600 4350 60  0000 C CNN
+F 2 "LEDs:LED-0805" H 6600 4350 60  0001 C CNN
 F 3 "" H 6600 4350 60  0000 C CNN
 	1    6600 4350
@@
 $EndComp
 $Comp
-L VCC #PWR?
+L VCC #PWR018
 U 1 1 559331B7
 P 6600 4050
-F 0 "#PWR?" H 6600 3900 50  0001 C CNN
+F 0 "#PWR018" H 6600 3900 50  0001 C CNN
 F 1 "VCC" H 6600 4200 50  0000 C CNN
 F 2 "" H 6600 4050 60  0000 C CNN
@@
 $EndComp
 $Comp
-L R R?
+L R R2
 U 1 1 559331E9
 P 6600 4800
-F 0 "R?" V 6680 4800 50  0000 C CNN
+F 0 "R2" V 6680 4800 50  0000 C CNN
 F 1 "R" V 6600 4800 50  0000 C CNN
 F 2 "Resistors_SMD:R_0805" V 6530 4800 30  0001 C CNN
@@
 	6600 4550 6600 4650
 $Comp
-L GND #PWR?
+L GND #PWR019
 U 1 1 559333A4
 P 6600 5000
-F 0 "#PWR?" H 6600 4750 50  0001 C CNN
+F 0 "#PWR019" H 6600 4750 50  0001 C CNN
 F 1 "GND" H 6600 4850 50  0000 C CNN
 F 2 "" H 6600 5000 60  0000 C CNN
