File: rxfe_mcm/usrp_io.sch (KiCad schematic (older format))
At the start: 24 parts, among them J201 DB15, P201 CONN_02X10, U202 CONN_SMA, U203 74HC04_FULL, U204 CONN_SMA, U205 ADP7158, U206 CONN_SMA, U209 CONN_SMA

Commit message: removed tx path amp, erc fixes
Connections:
- no-connect marks 1 -> 6
Changed lines of the file:
@@
 LIBS:adp7158
 LIBS:pe4312
+LIBS:isl3295efhz-t
 LIBS:rxfe_mcm-cache
 EELAYER 25 0
@@
 $EndComp
 $Comp
-L GND #PWR223
+L GND #PWR01
 U 1 1 59826F34
 P 13700 4500
-F 0 "#PWR223" H 13700 4250 50  0001 C CNN
+F 0 "#PWR01" H 13700 4250 50  0001 C CNN
 F 1 "GND" H 13700 4350 50  0000 C CNN
 F 2 "" H 13700 4500 50  0000 C CNN
@@
 AMPB2_CTRL
 $Comp
-L GND #PWR214
+L GND #PWR02
 U 1 1 5982BDE0
 P 12250 5450
-F 0 "#PWR214" H 12250 5200 50  0001 C CNN
+F 0 "#PWR02" H 12250 5200 50  0001 C CNN
 F 1 "GND" H 12250 5300 50  0000 C CNN
 F 2 "" H 12250 5450 50  0000 C CNN
@@
 $EndComp
 $Comp
-L GND #PWR226
+L GND #PWR03
 U 1 1 598D7D01
 P 14100 4500
-F 0 "#PWR226" H 14100 4250 50  0001 C CNN
+F 0 "#PWR03" H 14100 4250 50  0001 C CNN
 F 1 "GND" H 14100 4350 50  0000 C CNN
 F 2 "" H 14100 4500 50  0000 C CNN
@@
 $EndComp
 $Comp
-L +3V3 #PWR209
+L +3V3 #PWR04
 U 1 1 598DD83D
 P 11550 6850
-F 0 "#PWR209" H 11550 6700 50  0001 C CNN
+F 0 "#PWR04" H 11550 6700 50  0001 C CNN
 F 1 "+3V3" H 11550 6990 50  0000 C CNN
 F 2 "" H 11550 6850 50  0000 C CNN
@@
 $EndComp
 $Comp
-L VPP #PWR227
+L VPP #PWR05
 U 1 1 59903DFA
 P 14250 6850
-F 0 "#PWR227" H 14250 6700 50  0001 C CNN
+F 0 "#PWR05" H 14250 6700 50  0001 C CNN
 F 1 "VPP" H 14250 7000 50  0000 C CNN
 F 2 "" H 14250 6850 50  0000 C CNN
@@
 $EndComp
 $Comp
-L GND #PWR219
+L GND #PWR06
 U 1 1 599045BA
 P 13450 7950
-F 0 "#PWR219" H 13450 7700 50  0001 C CNN
+F 0 "#PWR06" H 13450 7700 50  0001 C CNN
 F 1 "GND" H 13450 7800 50  0000 C CNN
 F 2 "" H 13450 7950 50  0000 C CNN
@@
 $EndComp
 $Comp
-L GND #PWR224
+L GND #PWR07
 U 1 1 59904683
 P 13850 7950
-F 0 "#PWR224" H 13850 7700 50  0001 C CNN
+F 0 "#PWR07" H 13850 7700 50  0001 C CNN
 F 1 "GND" H 13850 7800 50  0000 C CNN
 F 2 "" H 13850 7950 50  0000 C CNN
@@
 $EndComp
 $Comp
-L GND #PWR228
+L GND #PWR08
 U 1 1 599046FD
 P 14250 7950
-F 0 "#PWR228" H 14250 7700 50  0001 C CNN
+F 0 "#PWR08" H 14250 7700 50  0001 C CNN
 F 1 "GND" H 14250 7800 50  0000 C CNN
 F 2 "" H 14250 7950 50  0000 C CNN
@@
 $EndComp
 $Comp
-L GND #PWR211
+L GND #PWR09
 U 1 1 599050DD
 P 11850 7950
-F 0 "#PWR211" H 11850 7700 50  0001 C CNN
+F 0 "#PWR09" H 11850 7700 50  0001 C CNN
 F 1 "GND" H 11850 7800 50  0000 C CNN
 F 2 "" H 11850 7950 50  0000 C CNN
@@
 $EndComp
 $Comp
-L GND #PWR210
+L GND #PWR010
 U 1 1 5990515D
 P 11550 7950
-F 0 "#PWR210" H 11550 7700 50  0001 C CNN
+F 0 "#PWR010" H 11550 7700 50  0001 C CNN
 F 1 "GND" H 11550 7800 50  0000 C CNN
 F 2 "" H 11550 7950 50  0000 C CNN
@@
 $EndComp
 $Comp
-L GND #PWR217
+L GND #PWR011
 U 1 1 59905965
 P 12700 7950
-F 0 "#PWR217" H 12700 7700 50  0001 C CNN
+F 0 "#PWR011" H 12700 7700 50  0001 C CNN
 F 1 "GND" H 12700 7800 50  0000 C CNN
 F 2 "" H 12700 7950 50  0000 C CNN
@@
 $EndComp
 $Comp
-L VPP #PWR212
+L VPP #PWR012
 U 1 1 5990693F
 P 12050 7750
-F 0 "#PWR212" H 12050 7600 50  0001 C CNN
+F 0 "#PWR012" H 12050 7600 50  0001 C CNN
 F 1 "VPP" H 12050 7900 50  0000 C CNN
 F 2 "" H 12050 7750 50  0000 C CNN
@@
 $EndComp
 $Comp
-L +3V3 #PWR222
+L +3V3 #PWR013
 U 1 1 5991D035
 P 13700 3800
-F 0 "#PWR222" H 13700 3650 50  0001 C CNN
+F 0 "#PWR013" H 13700 3650 50  0001 C CNN
 F 1 "+3V3" H 13700 3940 50  0000 C CNN
 F 2 "" H 13700 3800 50  0000 C CNN
@@
 $EndComp
 $Comp
-L GND #PWR204
+L GND #PWR014
 U 1 1 5983E2EE
 P 3300 10500
-F 0 "#PWR204" H 3300 10250 50  0001 C CNN
+F 0 "#PWR014" H 3300 10250 50  0001 C CNN
 F 1 "GND" H 3300 10350 50  0000 C CNN
 F 2 "" H 3300 10500 50  0000 C CNN
@@
 $EndComp
 $Comp
-L GND #PWR203
+L GND #PWR015
 U 1 1 5983EAFB
 P 3300 9300
-F 0 "#PWR203" H 3300 9050 50  0001 C CNN
+F 0 "#PWR015" H 3300 9050 50  0001 C CNN
 F 1 "GND" H 3300 9150 50  0000 C CNN
 F 2 "" H 3300 9300 50  0000 C CNN
@@
 $EndComp
 $Comp
-L GND #PWR202
+L GND #PWR016
 U 1 1 5983ED3F
 P 3300 7900
-F 0 "#PWR202" H 3300 7650 50  0001 C CNN
+F 0 "#PWR016" H 3300 7650 50  0001 C CNN
 F 1 "GND" H 3300 7750 50  0000 C CNN
 F 2 "" H 3300 7900 50  0000 C CNN
@@
 $EndComp
 $Comp
-L GND #PWR201
+L GND #PWR017
 U 1 1 5983ED56
 P 3300 6700
-F 0 "#PWR201" H 3300 6450 50  0001 C CNN
+F 0 "#PWR017" H 3300 6450 50  0001 C CNN
 F 1 "GND" H 3300 6550 50  0000 C CNN
 F 2 "" H 3300 6700 50  0000 C CNN
@@
 TR
 $Comp
-L GND #PWR206
+L GND #PWR018
 U 1 1 5986664A
 P 3350 1400
-F 0 "#PWR206" H 3350 1150 50  0001 C CNN
+F 0 "#PWR018" H 3350 1150 50  0001 C CNN
 F 1 "GND" H 3350 1250 50  0000 C CNN
 F 2 "" H 3350 1400 50  0000 C CNN
@@
 $EndComp
 $Comp
-L GND #PWR205
+L GND #PWR019
 U 1 1 598666AA
 P 3350 1200
-F 0 "#PWR205" H 3350 950 50  0001 C CNN
+F 0 "#PWR019" H 3350 950 50  0001 C CNN
 F 1 "GND" H 3350 1050 50  0000 C CNN
 F 2 "" H 3350 1200 50  0000 C CNN
@@
 TR
 $Comp
-L +3V3 #PWR220
+L +3V3 #PWR020
 U 1 1 59D4367C
 P 13500 1200
-F 0 "#PWR220" H 13500 1050 50  0001 C CNN
+F 0 "#PWR020" H 13500 1050 50  0001 C CNN
 F 1 "+3V3" H 13500 1340 50  0000 C CNN
 F 2 "" H 13500 1200 50  0000 C CNN
@@
 $EndComp
 $Comp
-L GND #PWR221
+L GND #PWR021
 U 1 1 59D437EF
 P 13500 2700
-F 0 "#PWR221" H 13500 2450 50  0001 C CNN
+F 0 "#PWR021" H 13500 2450 50  0001 C CNN
 F 1 "GND" H 13500 2550 50  0000 C CNN
 F 2 "" H 13500 2700 50  0000 C CNN
@@
 $EndComp
 $Comp
-L GND #PWR225
+L GND #PWR022
 U 1 1 59D43EF5
 P 13900 2700
-F 0 "#PWR225" H 13900 2450 50  0001 C CNN
+F 0 "#PWR022" H 13900 2450 50  0001 C CNN
 F 1 "GND" H 13900 2550 50  0000 C CNN
 F 2 "" H 13900 2700 50  0000 C CNN
@@
 $EndComp
 $Comp
-L GND #PWR213
+L GND #PWR023
 U 1 1 59D456DE
 P 12100 2700
-F 0 "#PWR213" H 12100 2450 50  0001 C CNN
+F 0 "#PWR023" H 12100 2450 50  0001 C CNN
 F 1 "GND" H 12100 2550 50  0000 C CNN
 F 2 "" H 12100 2700 50  0000 C CNN
@@
 $EndComp
 $Comp
-L GND #PWR215
+L GND #PWR024
 U 1 1 59D4591A
 P 12400 2700
-F 0 "#PWR215" H 12400 2450 50  0001 C CNN
+F 0 "#PWR024" H 12400 2450 50  0001 C CNN
 F 1 "GND" H 12400 2550 50  0000 C CNN
 F 2 "" H 12400 2700 50  0000 C CNN
@@
 $EndComp
 $Comp
-L GND #PWR216
+L GND #PWR025
 U 1 1 59D45B9A
 P 12700 2700
-F 0 "#PWR216" H 12700 2450 50  0001 C CNN
+F 0 "#PWR025" H 12700 2450 50  0001 C CNN
 F 1 "GND" H 12700 2550 50  0000 C CNN
 F 2 "" H 12700 2700 50  0000 C CNN
@@
 $EndComp
 $Comp
-L GND #PWR218
+L GND #PWR026
 U 1 1 59D45C8C
 P 13000 2700
-F 0 "#PWR218" H 13000 2450 50  0001 C CNN
+F 0 "#PWR026" H 13000 2450 50  0001 C CNN
 F 1 "GND" H 13000 2550 50  0000 C CNN
 F 2 "" H 13000 2700 50  0000 C CNN
@@
 $EndComp
 $Comp
-L GND #PWR207
+L GND #PWR027
 U 1 1 59D79E54
 P 4350 4450
-F 0 "#PWR207" H 4350 4200 50  0001 C CNN
+F 0 "#PWR027" H 4350 4200 50  0001 C CNN
 F 1 "GND" H 4350 4300 50  0000 C CNN
 F 2 "" H 4350 4450 50  0000 C CNN
@@
 $EndComp
 $Comp
-L GND #PWR208
+L GND #PWR028
 U 1 1 59D7B2F2
 P 5000 4450
-F 0 "#PWR208" H 5000 4200 50  0001 C CNN
+F 0 "#PWR028" H 5000 4200 50  0001 C CNN
 F 1 "GND" H 5000 4300 50  0000 C CNN
 F 2 "" H 5000 4450 50  0000 C CNN
@@
 Text Notes 4550 2950 0    59   ~ 0
 TODO: use net names instead of wiring.. this is messy
+NoConn ~ 4950 4000
+NoConn ~ 4950 4100
+NoConn ~ 4950 4200
+NoConn ~ 4450 4000
+NoConn ~ 4450 4100
 $EndSCHEMATC
