File: rxfe_mcm/rf_path.sch (KiCad schematic (older format))
At the start: 94 parts, among them J401 RF_SHIELD_TWO_PIECES, U401 TRF37B73, U402 MASW-007935-TR3000, U403 MASW-007935-TR3000, U404 TRF37B73, U405 SCLF-25, U406 SMP1330-005LF, U407 SMP1330-005LF, U408 MASW-007935-TR3000, U409 TRF37B73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

Commit message: moved limiter diode to fix short
Parts:
- R404: value 51 -> 60.4
- R405: value 2.4k -> 2k
- R411: value JMP -> DNP
Connections:
- net at C417.1, C516.2, L405.1: now also U516.3 (LIM)
- net at C417.2, L402.2, U404.7 (RFOUT): no longer U516.3 (LIM)
Other:
- moved on the sheet: U416
Changed lines of the file:
@@
 AR Path="/598253CB/5990C48F" Ref="R505"  Part="1"
 F 0 "R405" H 3280 10420 50  0000 L CNN
-F 1 "2.4k" H 3280 10360 50  0000 L CNN
+F 1 "2k" H 3280 10360 50  0000 L CNN
 F 2 "Resistors_SMD:R_0603" H 3250 10400 50  0001 C CNN
 F 3 "" H 3250 10400 50  0000 C CNN
@@
 AR Path="/598253CB/5990CA51" Ref="R504"  Part="1"
 F 0 "R404" H 3480 10220 50  0000 L CNN
-F 1 "51" H 3480 10160 50  0000 L CNN
+F 1 "60.4" H 3480 10160 50  0000 L CNN
 F 2 "Resistors_SMD:R_0603" H 3450 10200 50  0001 C CNN
 F 3 "" H 3450 10200 50  0000 C CNN
@@
 AR Path="/598253CB/59D56903" Ref="R511"  Part="1"
 F 0 "R411" H 15330 2820 50  0000 L CNN
-F 1 "JMP" H 15330 2760 50  0000 L CNN
+F 1 "DNP" H 15330 2760 50  0000 L CNN
 F 2 "Resistors_SMD:R_0603" H 15300 2800 50  0001 C CNN
 F 3 "" H 15300 2800 50  0000 C CNN
@@
 L SMP1330-005LF U516
 U 1 1 59D653DC
-P 14850 2900
+P 14000 1250
 AR Path="/598253CB/59D653DC" Ref="U516"  Part="1"
 AR Path="/597F80E0/59D653DC" Ref="U416"  Part="1"
-F 0 "U416" V 14450 2700 60  0000 C CNN
-F 1 "SMP1330-005LF" V 14550 2900 60  0000 C CNN
-F 2 "TO_SOT_Packages_SMD:SOT-23" H 14850 2900 60  0001 C CNN
-F 3 "" H 14850 2900 60  0000 C CNN
-	1    14850 2900
-	1    0    0    -1
+F 0 "U416" V 13600 1050 60  0000 C CNN
+F 1 "SMP1330-005LF" V 13700 1250 60  0000 C CNN
+F 2 "TO_SOT_Packages_SMD:SOT-23" H 14000 1250 60  0001 C CNN
+F 3 "" H 14000 1250 60  0000 C CNN
+	1    14000 1250
+	1    0    0    1
 $EndComp
 $Comp
 L GND #PWR0241
 U 1 1 59D653E2
-P 14750 3500
+P 13900 650
 AR Path="/598253CB/59D653E2" Ref="#PWR0241"  Part="1"
 AR Path="/597F80E0/59D653E2" Ref="#PWR0159"  Part="1"
-F 0 "#PWR0159" H 14750 3250 50  0001 C CNN
-F 1 "GND" H 14750 3350 50  0000 C CNN
-F 2 "" H 14750 3500 50  0000 C CNN
-F 3 "" H 14750 3500 50  0000 C CNN
-	1    14750 3500
-	-1   0    0    -1
+F 0 "#PWR0159" H 13900 400 50  0001 C CNN
+F 1 "GND" H 13900 500 50  0000 C CNN
+F 2 "" H 13900 650 50  0000 C CNN
+F 3 "" H 13900 650 50  0000 C CNN
+	1    13900 650
+	-1   0    0    1
 $EndComp
 $Comp
 L GND #PWR0242
 U 1 1 59D653E8
-P 14950 3500
+P 14100 650
 AR Path="/598253CB/59D653E8" Ref="#PWR0242"  Part="1"
 AR Path="/597F80E0/59D653E8" Ref="#PWR0160"  Part="1"
-F 0 "#PWR0160" H 14950 3250 50  0001 C CNN
-F 1 "GND" H 14950 3350 50  0000 C CNN
-F 2 "" H 14950 3500 50  0000 C CNN
-F 3 "" H 14950 3500 50  0000 C CNN
-	1    14950 3500
-	-1   0    0    -1
+F 0 "#PWR0160" H 14100 400 50  0001 C CNN
+F 1 "GND" H 14100 500 50  0000 C CNN
+F 2 "" H 14100 650 50  0000 C CNN
+F 3 "" H 14100 650 50  0000 C CNN
+	1    14100 650
+	-1   0    0    1
 $EndComp
 Text Notes 15550 750  0    118  ~ 0
@@
 	13350 2200 13650 2200
 Wire Wire Line
-	14000 2200 14000 2350
+	14000 1750 14000 2350
 Wire Wire Line
 	14000 2650 14000 2550
@@
 	5400 14150 5400 14350
 Wire Wire Line
-	14750 3500 14750 3400
-Wire Wire Line
-	14950 3500 14950 3400
-Wire Wire Line
-	14850 2400 14850 2200
-Connection ~ 14850 2200
+	13900 650  13900 750
+Wire Wire Line
+	14100 650  14100 750
 Wire Wire Line
 	3250 9100 3250 9650

Commit message: Replaced Obsolete Attenuator, added Docs
Parts:
- removed C452: 22 nF, Capacitors_SMD:C_0603, symbol C_Small
- removed U413: PE4312, Housings_DFN_QFN:QFN-20-1EP_4x4mm_Pitch0.5mm, symbol PE4312
- added U513: idtf1912ncgi, symbol idtf1912ncgi
Connections:
- net +3V3: now also U513.13 (VMODE), U513.6 (VDD)
- net ATT_LE: now also U513.5 (LE)
- net ATT_SCK: now also U513.4 (CLK)
- net ATT_SDI: now also U513.3 (DATA)
- net GND: now also U513.1 (D5), U513.10 (GND), U513.11 (GND), U513.12 (GND), U513.15 (D4), U513.16 (D3), U513.17 (D2), U513.18 (GND), U513.19 (D1), U513.20 (D0)
- net at C440.2: now also U513.2 (RF1)
- net at C511.2: now also U513.14 (RF2)
Other:
- note added: "In Serial Mode"
- note removed: "set power-on attenuation with C0.5 to C16\ncurrently configured for 16 dB"
- moved on the sheet: C451

Commit message: updated refe_mcm and made documentation
Parts:
- U513: footprint (none) -> Housings_DFN_QFN:QFN-20-1EP_4x4mm_Pitch0.5mm
Connections:
- net GND: now also U513.21 (EPAD)
